File: BSPD 27/BSPD 27.kicad_pcb (KiCad board)
At the start: 2 copper layers, 37 parts, among them Q1 Q_NMOS_GSD, U1 TLV9032DGKR, U10 74AHC1G32, U2 TLV9032DGKR, U3 TLV9032DGKR, U4 Optocoupler, U5 Inverter_Schmitt_Dual, U6 74AHC1G32, U7 74AHC1G00, U8 SN74AHC1G08DBVR, U9 SN74AHC1G08DBVR

Commit message: Mostly Order ready BSPD and FL
Parts:
- removed D1: SD05.TCT, Diode_SMD:D_SOD-323
- added H1: MountingHole, MountingHole:MountingHole_3.2mm_M3_DIN965_Pad, F.Cu at (135.6, 102.6)
- added H2: MountingHole, MountingHole:MountingHole_3.2mm_M3_DIN965_Pad, F.Cu at (170.5, 102.6)
- added J1: Conn_01x04_Pin, 1.Custom:SAMTEC_TSW-104-07-L-S, B.Cu at (153.8, 94.2)
- added J2: Conn_01x04_Pin, 1.Custom:SAMTEC_TSW-104-07-L-S, B.Cu at (153.8, 110.6)
- C1, C2, C3: footprint Capacitor_SMD:C_1206_3216Metric -> Capacitor_SMD:C_0603_1608Metric
- C10, C11, C4, C5, C6, C7, C8, C9: footprint Capacitor_SMD:C_1206_3216Metric -> Capacitor_SMD:C_0603_1608Metric; moved to B.Cu
- R5: value 70k -> 69.8k; moved to B.Cu
- R6: moved to B.Cu
- R7: value 400k -> 340k
- U5: value Inverter_Schmitt_Dual -> SN74LVC2G17MDCKREP
- moved C1 34.4 mm to (164.0, 103.2), turned to 180 degrees
- moved U9 32.8 mm to (159.5, 100.6), turned to 90 degrees
- moved U10 30.6 mm to (156.5, 100.6), turned to 90 degrees
- moved C6 27.6 mm to (157.8, 98.8)
- moved U5 27.4 mm to (153.7, 97.2), turned to 180 degrees
- moved R1 27.3 mm to (169.5, 109.1)
- moved U7 26.7 mm to (153.5, 100.7), turned to 90 degrees
- moved R2 25.4 mm to (167.8, 111.0)
- moved C3 25.4 mm to (156.6, 103.2), turned to 180 degrees
- moved U8 23.6 mm to (150.6, 100.7), turned to 90 degrees
- moved U6 23.2 mm to (150.0, 97.2), turned to 180 degrees
- moved C10 22.7 mm to (160.2, 100.7), turned to 90 degrees
- moved Q1 22.3 mm to (137.1, 96.8), turned to 180 degrees
- moved R5 22.0 mm to (155.1, 99.8), turned to 90 degrees
- moved TP1 21.1 mm to (170.0, 97.4)
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Routing:
- net +5V: track 0.00 -> 111.8 mm, vias 0 -> 12
- net /0.385V: track 0.00 -> 30.8 mm, vias 0 -> 4
- net /THRESH_BSE: track 0.00 -> 24.7 mm, vias 0 -> 3
- net BSPD_OUT: track 0.00 -> 19.8 mm, vias 0 -> 1
- net /ACCUM_V: track 0.00 -> 19.4 mm, vias 0 -> 2
- net +12V: track 0.00 -> 17.8 mm
- net /BSE_2: track 0.00 -> 16.4 mm
- net /THRESH_ACCUM: track 0.00 -> 16.3 mm, vias 0 -> 3
- net /BSE_1: track 0.00 -> 15.4 mm
- net Net-(U1-Pad1): track 0.00 -> 11.2 mm, vias 0 -> 2
- net Net-(U1-Pad7): track 0.00 -> 9.24 mm, vias 0 -> 2
- net Net-(U10-Pad1): track 0.00 -> 6.61 mm
- net Net-(Q1-G): track 0.00 -> 6.41 mm
- net Net-(U3-Pad1): track 0.00 -> 5.51 mm, vias 0 -> 2
- net Net-(U10-Pad2): track 0.00 -> 5.45 mm
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- added copper zone on B.Cu, net GND
- added copper zone on F.Cu, net GND
- added copper zone on B.Cu, net GNDPWR
- added copper zone on F.Cu, net GNDPWR
Other:
- board outline added: 43.1 x 20.7 mm

Commit message: V1 of BSPD FL and Power ready for order
Parts:
- removed the U5 at (153.7, 97.2)
- added G***: LOGO, LOGO, B.Cu at (163.6, 107.9)
- added G***: LOGO, LOGO, B.Cu at (155.4, 106.5)
- added U4: SN74LVC2G17MDCKREP, Package_TO_SOT_SMD:SOT-363_SC-70-6, F.Cu at (153.7, 97.2)
- C6, C7: footprint Capacitor_SMD:C_0603_1608Metric -> Capacitor_SMD:C_0805_2012Metric
- moved C7 3.40 mm to (160.2, 97.2), turned to 90 degrees
- moved C6 1.26 mm to (157.8, 97.5), turned to 90 degrees
- renumbered U4 to U5
Routing:
- net Net-(C7-Pad1): track 4.19 -> 8.37 mm
- net +5V: track 111.8 -> 112.8 mm
Other:
- board text added: "TR27 BSPD"
