File: BSPD 27/BSPD 27.kicad_sch (KiCad schematic)
At the start: 37 parts, among them Q1 Q_NMOS_GSD, U1 TLV9032DGKR, U10 74AHC1G32, U2 TLV9032DGKR, U3 TLV9032DGKR, U4 Optocoupler, U5 Inverter_Schmitt_Dual, U6 74AHC1G32, U7 74AHC1G00, U8 SN74AHC1G08DBVR, U9 SN74AHC1G08DBVR

Commit message: Mostly Order ready BSPD and FL
Parts:
- removed D1: SD05.TCT, Diode_SMD:D_SOD-323, symbol Diode:PTVS5V0Z1USK
- added H1, H2: MountingHole, MountingHole:MountingHole_3.2mm_M3_DIN965_Pad, symbol Mechanical:MountingHole
- added J1, J2: Conn_01x04_Pin, 1.Custom:SAMTEC_TSW-104-07-L-S, symbol Connector:Conn_01x04_Pin
- C1, C10, C11, C2, C3, C4, C5, C6, C7, C8, C9: footprint Capacitor_SMD:C_1206_3216Metric -> Capacitor_SMD:C_0603_1608Metric
- R5: value 70k -> 69.8k
- R7: value 400k -> 340k
- U5: value Inverter_Schmitt_Dual -> SN74LVC2G17MDCKREP
Connections:
- net +12V: now also J1.3 (Pin_3)
- net +5V: now also J1.4 (Pin_4)
- net ACCUM_V: now also J2.4 (Pin_4)
- net BSE_1: now also J2.2 (Pin_2)
- net BSE_2: now also J2.3 (Pin_3)
- net BSPD_OUT: now also J1.2 (Pin_2)
- net GND: now also J2.1 (Pin_1)
- net GNDPWR: now also J1.1 (Pin_1)
- no-connect marks 1 -> 0
Other:
- note added: "τ = 0.0698s 1.427τ =~ 0.1s"
- note added: "τ = 0.34s 1.427τ = 0.485s"
- note removed: "12v supply from battery for fault latch"
- note removed: "5V"
- note removed: "5v supply isolated from VCU"
- note removed: "BSE Voltage (0.5-4.5V)"
- note removed: "GND"
- note removed: "NC"
- note removed: "OUT"
- note removed: "τ = 0.07s 1.427τ = 0.1"
- note removed: "τ = 0.4s 1.427τ = 0.485s"

Commit message: V1 of BSPD FL and Power ready for order
Parts:
- removed U5: SN74LVC2G17MDCKREP, Package_TO_SOT_SMD:SOT-363_SC-70-6, symbol 74xGxx:Inverter_Schmitt_Dual
- added U4: SN74LVC2G17MDCKREP, Package_TO_SOT_SMD:SOT-363_SC-70-6, symbol 74xGxx:74LVC2G17
- C6, C7: footprint Capacitor_SMD:C_0603_1608Metric -> Capacitor_SMD:C_0805_2012Metric
- renumbered U4 to U5
Connections:
- net +5V: now also U4.5 (VCC)
- net GND: now also U4.2 (GND)
- net at C7.1, R7.2: now also U4.3
- net at C6.1, R5.2: now also U4.1
- net at U6.2: now also U4.4
- net at U6.1: now also U4.6
Other:
- moved on the sheet: C4

Commit message: added mouser# & digikey# to all components
Parts:
- C1, C10, C11, C2, C3, C4, C5, C8, C9: Digikey# (none) -> 587-MCAST168SB5104KTNA01CT-ND; MF# (none) -> MCAST168SB5104KTNA01; Mouser# (none) -> 963-MCAST168SB5104KT
- C6, C7: Digikey# (none) -> 13-AC0805KKX7R9BB105CT-ND; MF# (none) -> AC0805KKX7R9BB105; Mouser# (none) -> 603-AC0805KKX7R9B105
- J1, J2: Digikey# (none) -> N/A; MF# (none) -> N/A; Mouser# (none) -> N/A
- Q1: Mouser# 637-MMFTN6001 -> 637-MMFTN6001
- R1: Digikey# (none) -> 2019-RK73H2ATTD1202FCT-ND; MF# (none) -> RK73H2ATTD1202F; Mouser# (none) -> 660-RK73H2ATTD1202F
- R10, R8, R9: Digikey# (none) -> 13-RC0805FR-10100KLCT-ND; MF# (none) -> RC0805FR-10100KL; Mouser# (none) -> 603-RC0805FR-10100KL
- R2, R6: Digikey# (none) -> 311-1.00KCRCT-ND; MF# (none) -> RC0805FR-071KL; Mouser# (none) -> 603-RC0805FR-071KL
- R3, R4: Digikey# (none) -> 311-10.0KCRCT-ND; MF# (none) -> RC0805FR-0710KL; Mouser# (none) -> 603-RC0805FR-0710KL
- R5: Digikey# (none) -> 408-RR1220P-6982-D-MCT-ND; MF# (none) -> RR1220P-6982-D-M; Mouser# (none) -> 754-RR1220P-6982D-M
- R7: Digikey# (none) -> 13-AC0805FR-07340KLTR-ND; MF# (none) -> AC0805FR-07340KL; Mouser# (none) -> 603-AC0805FR-07340KL
- RV1, RV2: Digikey# (none) -> PVG5A103C03B00-ND; MF# (none) -> PVG5A103C03B00; Mouser# (none) -> 81-PVG5A103C03B00
- U1, U2, U3: Digikey# (none) -> 296-TLV9032DGKRCT-ND; MF# (none) -> TLV9032DGKR; Mouser# (none) -> 595-TLV9032DGKR
- U10, U6: Digikey# (none) -> 296-9848-1-ND; MF# (none) -> SN74LVC1G32DCKR; Mouser# (none) -> 595-SN74LVC1G32DCKR
- U4: Digikey# (none) -> 296-22358-1-ND; MF# (none) -> SN74LVC2G17MDCKREP; Mouser# (none) -> 595-SN74L2G17MDCKREP
- U5: Mouser# 78-VOS617A-3T -> 78-VOS617A-3T
- U7: Digikey# (none) -> 296-9846-1-ND; MF# (none) -> SN74LVC1G00DCKR; Mouser# (none) -> 595-SN74LVC1G00DCKR
- U8, U9: Digikey# (none) -> 296-18066-1-ND; MF# (none) -> SN74LVC1G11DCKR; Mouser# (none) -> 595-SN74LVC1G11DCKR

Commit message: fixed bspd and gate part #
Parts:
- U8: MF# SN74LVC1G11DCKR -> SN74LVC1G08DCKR; Mouser# 595-SN74LVC1G11DCKR -> 595-SN74LVC1G08DCKR
Changed lines of the file:
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@@
 			)
 		)
-		(property "MF#" "SN74LVC1G11DCKR  "
+		(property "MF#" "SN74LVC1G08DCKR"
 			(at 100.33 182.88 0)
 			(hide yes)
@@
 			)
 		)
-		(property "Mouser#" "595-SN74LVC1G11DCKR "
+		(property "Mouser#" "595-SN74LVC1G08DCKR"
 			(at 100.33 182.88 0)
 			(hide yes)
