File: BSPD 27/BSPD 27.kicad_sch (KiCad schematic)
At the start: 40 parts, among them J1 Conn_01x04_Pin, J2 Conn_01x04_Pin, Q1 Q_NMOS_GSD, U1 TLV9032DGKR, U10 74AHC1G32, U2 TLV9032DGKR, U3 TLV9032DGKR, U4 SN74LVC2G17MDCKREP, U5 Optocoupler, U6 74AHC1G32, U7 74AHC1G00, U8 SN74AHC1G08DBVR, U9 SN74AHC1G08DBVR

Commit message: fixed part # on bspd and fl
Parts:
- C1, C10, C11, C2, C3, C4, C5, C8, C9: Digikey# 587-MCAST168SB5104KTNA01CT-ND -> (none); MF# MCAST168SB5104KTNA01 -> 311-3034-2-ND; Mouser# 963-MCAST168SB5104KT -> AC0603KRX7R9BB104
- C6, C7: Digikey# 13-AC0805KKX7R9BB105CT-ND -> (none); MF# AC0805KKX7R9BB105 -> 13-AC0805KKX7R9BB105CT-ND; Mouser# 603-AC0805KKX7R9B105 -> AC0805KKX7R9BB105
- Q1: Digikey# 4878-MMFTN6001TR-ND -> (none)
- R1: Digikey# 2019-RK73H2ATTD1202FCT-ND -> 2019-RK73H2ATTD1202FCT-ND; Mouser# 660-RK73H2ATTD1202F -> (none)
- R10, R8, R9: Mouser# 603-RC0805FR-10100KL -> (none)
- R2, R6: Mouser# 603-RC0805FR-071KL -> (none)
- R3, R4: Mouser# 603-RC0805FR-0710KL -> (none)
- R5: Mouser# 754-RR1220P-6982D-M -> (none)
- R7: Mouser# 603-AC0805FR-07340KL -> (none)
- RV1, RV2: Digikey# PVG5A103C03B00-ND -> (none)
- U1, U2, U3: Mouser# 595-TLV9032DGKR -> (none)
- U10, U6: Digikey# 296-9848-1-ND -> (none)
- U4: Mouser# 595-SN74L2G17MDCKREP -> (none)
- U5: Digikey# VOS617A-3TTR-ND -> 78-VOS617A-3T; Mouser# 78-VOS617A-3T -> (none)
- U7: Digikey# 296-9846-1-ND -> (none)
- U8, U9: Digikey# 296-18066-1-ND -> (none)
Changed lines of the file:
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@@
 			)
 		)
-		(property "Digikey#" "587-MCAST168SB5104KTNA01CT-ND"
+		(property "Digikey#" ""
 			(at 300.99 198.12 90)
 			(hide yes)
@@
 			)
 		)
-		(property "MF#" "MCAST168SB5104KTNA01"
+		(property "MF#" "311-3034-2-ND "
 			(at 300.99 198.12 90)
 			(hide yes)
@@
 			)
 		)
-		(property "Mouser#" "963-MCAST168SB5104KT"
+		(property "Mouser#" "AC0603KRX7R9BB104  "
 			(at 300.99 198.12 90)
 			(hide yes)
@@
 			)
 		)
-		(property "Digikey#" "296-9846-1-ND"
+		(property "Digikey#" ""
 			(at 152.4 154.94 0)
 			(hide yes)
@@
 			)
 		)
-		(property "Mouser#" "595-TLV9032DGKR"
+		(property "Mouser#" ""
 			(at 275.59 158.75 0)
 			(hide yes)
@@
 			)
 		)
-		(property "Digikey#" "296-9848-1-ND"
+		(property "Digikey#" ""
 			(at 308.61 213.36 0)
 			(hide yes)
@@
 			)
 		)
-		(property "Digikey#" "587-MCAST168SB5104KTNA01CT-ND"
+		(property "Digikey#" ""
 			(at 175.26 31.75 0)
 			(hide yes)
@@
 			)
 		)
-		(property "MF#" "MCAST168SB5104KTNA01"
+		(property "MF#" "311-3034-2-ND "
 			(at 175.26 31.75 0)
 			(hide yes)
@@
 			)
 		)
-		(property "Mouser#" "963-MCAST168SB5104KT"
+		(property "Mouser#" "AC0603KRX7R9BB104  "
 			(at 175.26 31.75 0)
 			(hide yes)
@@
 			)
 		)
-		(property "Digikey#" "296-18066-1-ND "
+		(property "Digikey#" ""
 			(at 100.33 182.88 0)
 			(hide yes)
@@
 			)
 		)
-		(property "Mouser#" "603-RC0805FR-0710KL "
+		(property "Mouser#" ""
 			(at 346.71 86.36 0)
 			(hide yes)
@@
 			)
 		)
-		(property "Mouser#" "603-RC0805FR-071KL  "
+		(property "Mouser#" ""
 			(at 323.85 90.17 0)
 			(hide yes)
@@
 			)
 		)
-		(property "Mouser#" "603-RC0805FR-10100KL"
+		(property "Mouser#" ""
 			(at 34.29 177.8 0)
 			(hide yes)
@@
 			)
 		)
-		(property "Mouser#" "595-SN74L2G17MDCKREP"
+		(property "Mouser#" ""
 			(at 269.24 90.17 0)
 			(hide yes)
@@
 			)
 		)
-		(property "Mouser#" "595-SN74L2G17MDCKREP"
+		(property "Mouser#" ""
 			(at 185.42 33.02 0)
 			(hide yes)
@@
 			)
 		)
-		(property "Digikey#" "296-18066-1-ND "
+		(property "Digikey#" ""
 			(at 356.87 185.42 0)
 			(hide yes)
@@
 			)
 		)
-		(property "Digikey#" "13-AC0805KKX7R9BB105CT-ND"
+		(property "Digikey#" ""
 			(at 247.65 118.11 0)
 			(hide yes)
@@
 			)
 		)
-		(property "MF#" "AC0805KKX7R9BB105 "
+		(property "MF#" "13-AC0805KKX7R9BB105CT-ND "
 			(at 247.65 118.11 0)
 			(hide yes)
@@
 			)
 		)
-		(property "Mouser#" "603-AC0805KKX7R9B105 "
+		(property "Mouser#" "AC0805KKX7R9BB105  "
 			(at 247.65 118.11 0)
 			(hide yes)
@@
 			)
 		)
-		(property "Mouser#" "603-RC0805FR-10100KL"
+		(property "Mouser#" ""
 			(at 34.29 138.43 0)
 			(hide yes)
@@
 			)
 		)
-		(property "Digikey#" "13-AC0805KKX7R9BB105CT-ND"
+		(property "Digikey#" ""
 			(at 247.65 95.25 0)
 			(hide yes)
@@
 			)
 		)
-		(property "MF#" "AC0805KKX7R9BB105 "
+		(property "MF#" "13-AC0805KKX7R9BB105CT-ND "
 			(at 247.65 95.25 0)
 			(hide yes)
@@
 			)
 		)
-		(property "Mouser#" "603-AC0805KKX7R9B105 "
+		(property "Mouser#" "AC0805KKX7R9BB105  "
 			(at 247.65 95.25 0)
 			(hide yes)
@@
 			)
 		)
-		(property "Mouser#" "603-RC0805FR-071KL  "
+		(property "Mouser#" ""
 			(at 351.79 40.64 0)
 			(hide yes)
@@
 			)
 		)
-		(property "Mouser#" "595-TLV9032DGKR"
+		(property "Mouser#" ""
 			(at 53.34 170.18 0)
 			(hide yes)
@@
 			)
 		)
-		(property "Mouser#" "595-TLV9032DGKR"
+		(property "Mouser#" ""
 			(at 250.19 30.48 0)
 			(hide yes)
@@
 			)
 		)
-		(property "Digikey#" "296-9848-1-ND"
+		(property "Digikey#" ""
 			(at 299.72 101.6 0)
 			(hide yes)
@@
 			)
 		)
-		(property "Digikey#" "4878-MMFTN6001TR-ND"
+		(property "Digikey#" ""
 			(at 353.06 96.52 0)
 			(hide yes)
@@
 			)
 		)
-		(property "Digikey#" "587-MCAST168SB5104KTNA01CT-ND"
+		(property "Digikey#" ""
 			(at 256.54 30.48 0)
 			(hide yes)
@@
 			)
 		)
-		(property "MF#" "MCAST168SB5104KTNA01"
+		(property "MF#" "311-3034-2-ND "
 			(at 256.54 30.48 0)
 			(hide yes)
@@
 			)
 		)
-		(property "Mouser#" "963-MCAST168SB5104KT"
+		(property "Mouser#" "AC0603KRX7R9BB104  "
 			(at 256.54 30.48 0)
 			(hide yes)
@@
 			)
 		)
-		(property "Digikey#" "587-MCAST168SB5104KTNA01CT-ND"
+		(property "Digikey#" ""
 			(at 350.52 170.18 90)
 			(hide yes)
@@
 			)
 		)
-		(property "MF#" "MCAST168SB5104KTNA01"
+		(property "MF#" "311-3034-2-ND "
 			(at 350.52 170.18 90)
 			(hide yes)
@@
 			)
 		)
-		(property "Mouser#" "963-MCAST168SB5104KT"
+		(property "Mouser#" "AC0603KRX7R9BB104  "
 			(at 350.52 170.18 90)
 			(hide yes)
@@
 			)
 		)
-		(property "Digikey#" "587-MCAST168SB5104KTNA01CT-ND"
+		(property "Digikey#" ""
 			(at 236.22 30.48 0)
 			(hide yes)
@@
 			)
 		)
-		(property "MF#" "MCAST168SB5104KTNA01"
+		(property "MF#" "311-3034-2-ND "
 			(at 236.22 30.48 0)
 			(hide yes)
@@
 			)
 		)
-		(property "Mouser#" "963-MCAST168SB5104KT"
+		(property "Mouser#" "AC0603KRX7R9BB104  "
 			(at 236.22 30.48 0)
 			(hide yes)
@@
 			)
 		)
-		(property "Mouser#" "603-RC0805FR-0710KL "
+		(property "Mouser#" ""
 			(at 355.6 86.36 0)
 			(hide yes)
@@
 			)
 		)
-		(property "Mouser#" "595-SN74L2G17MDCKREP"
+		(property "Mouser#" ""
 			(at 269.24 113.03 0)
 			(hide yes)
@@
 			)
 		)
-		(property "Mouser#" "78-VOS617A-3T "
+		(property "Mouser#" ""
 			(at 339.09 99.06 0)
 			(hide yes)
@@
 			)
 		)
-		(property "Digikey#" "VOS617A-3TTR-ND"
+		(property "Digikey#" " 78-VOS617A-3T "
 			(at 339.09 99.06 0)
 			(hide yes)
@@
 			)
 		)
-		(property "Digikey#" "  PVG5A103C03B00-ND"
+		(property "Digikey#" ""
 			(at 297.18 34.29 0)
 			(hide yes)
@@
 			)
 		)
-		(property "Mouser#" "595-TLV9032DGKR"
+		(property "Mouser#" ""
 			(at 53.34 213.36 0)
 			(hide yes)
@@
 			)
 		)
-		(property "Mouser#" "603-RC0805FR-10100KL"
+		(property "Mouser#" ""
 			(at 34.29 220.98 0)
 			(hide yes)
@@
 			)
 		)
-		(property "Mouser#" "595-TLV9032DGKR"
+		(property "Mouser#" ""
 			(at 275.59 232.41 0)
 			(hide yes)
@@
 			)
 		)
-		(property "Digikey#" "2019-RK73H2ATTD1202FCT-ND"
+		(property "Digikey#" "2019-RK73H2ATTD1202FCT-ND "
 			(at 351.79 30.48 0)
 			(hide yes)
@@
 			)
 		)
-		(property "Mouser#" "660-RK73H2ATTD1202F"
+		(property "Mouser#" ""
 			(at 351.79 30.48 0)
 			(hide yes)
@@
 			)
 		)
-		(property "Mouser#" "595-TLV9032DGKR"
+		(property "Mouser#" ""
 			(at 210.82 30.48 0)
 			(hide yes)
@@
 			)
 		)
-		(property "Mouser#" "603-AC0805FR-07340KL"
+		(property "Mouser#" ""
 			(at 240.03 113.03 90)
 			(hide yes)
@@
 			)
 		)
-		(property "Mouser#" "754-RR1220P-6982D-M"
+		(property "Mouser#" ""
 			(at 240.03 90.17 90)
 			(hide yes)
@@
 			)
 		)
-		(property "Digikey#" "587-MCAST168SB5104KTNA01CT-ND"
+		(property "Digikey#" ""
 			(at 217.17 30.48 0)
 			(hide yes)
@@
 			)
 		)
-		(property "MF#" "MCAST168SB5104KTNA01"
+		(property "MF#" "311-3034-2-ND "
 			(at 217.17 30.48 0)
 			(hide yes)
@@
 			)
 		)
-		(property "Mouser#" "963-MCAST168SB5104KT"
+		(property "Mouser#" "AC0603KRX7R9BB104  "
 			(at 217.17 30.48 0)
 			(hide yes)
@@
 			)
 		)
-		(property "Digikey#" "587-MCAST168SB5104KTNA01CT-ND"
+		(property "Digikey#" ""
 			(at 292.1 86.36 90)
 			(hide yes)
@@
 			)
 		)
-		(property "MF#" "MCAST168SB5104KTNA01"
+		(property "MF#" "311-3034-2-ND "
 			(at 292.1 86.36 90)
 			(hide yes)
@@
 			)
 		)
-		(property "Mouser#" "963-MCAST168SB5104KT"
+		(property "Mouser#" "AC0603KRX7R9BB104  "
 			(at 292.1 86.36 90)
 			(hide yes)
@@
 			)
 		)
-		(property "Digikey#" "587-MCAST168SB5104KTNA01CT-ND"
+		(property "Digikey#" ""
 			(at 144.78 139.7 90)
 			(hide yes)
@@
 			)
 		)
-		(property "MF#" "MCAST168SB5104KTNA01"
+		(property "MF#" "311-3034-2-ND "
 			(at 144.78 139.7 90)
 			(hide yes)
@@
 			)
 		)
-		(property "Mouser#" "963-MCAST168SB5104KT"
+		(property "Mouser#" "AC0603KRX7R9BB104  "
 			(at 144.78 139.7 90)
 			(hide yes)
@@
 			)
 		)
-		(property "Digikey#" "587-MCAST168SB5104KTNA01CT-ND"
+		(property "Digikey#" ""
 			(at 93.98 166.37 90)
 			(hide yes)
@@
 			)
 		)
-		(property "MF#" "MCAST168SB5104KTNA01"
+		(property "MF#" "311-3034-2-ND "
 			(at 93.98 166.37 90)
 			(hide yes)
@@
 			)
 		)
-		(property "Mouser#" "963-MCAST168SB5104KT"
+		(property "Mouser#" "AC0603KRX7R9BB104  "
 			(at 93.98 166.37 90)
 			(hide yes)
@@
 			)
 		)
-		(property "Mouser#" "595-TLV9032DGKR"
+		(property "Mouser#" ""
 			(at 229.87 30.48 0)
 			(hide yes)
@@
 			)
 		)
-		(property "Mouser#" "595-TLV9032DGKR"
+		(property "Mouser#" ""
 			(at 275.59 195.58 0)
 			(hide yes)
@@
 			)
 		)
-		(property "Mouser#" "595-TLV9032DGKR"
+		(property "Mouser#" ""
 			(at 53.34 130.81 0)
 			(hide yes)
@@
 			)
 		)
-		(property "Digikey#" "  PVG5A103C03B00-ND"
+		(property "Digikey#" ""
 			(at 330.2 34.29 0)
 			(hide yes)
