File: Fault Latch 27/Fault Latch 27.kicad_pcb (KiCad board)
At the start: 2 copper layers, 37.6 x 50.9 mm, 95 parts, among them J1 Conn_01x01_Pin, J2 Conn_01x01_Pin, J3 Conn_01x06_Pin, J4 Conn_01x06_Pin, J5 Conn_01x01_Pin, K1 OJ-SS-112LMH2, K2 OJ-SS-112LMH2, K3 OJ-SS-112LMH2, Q1 Q_NMOS_GSD, Q10 Q_NMOS_GSD, Q11 Q_NMOS_GSD, Q2 Q_NMOS_GSD, Q3 Q_NMOS_GSD, Q4 Q_NMOS_GSD, Q5 Q_NMOS_GSD, Q6 Q_NMOS_GSD, Q7 Q_NMOS_GSD, Q8 Q_NMOS_GSD, Q9 Q_NMOS_GSD, SW1 SW_Omron_B3FS, U1 D-Latch, U10 SN74AHC1G08DBVR, U11 D-Latch, U12 Optocoupler, U13 74AHC1G32, U2 Optocoupler, U3 74AHC1G32, U4 SN74AHC1G08DBVR, U5 D-Latch, U6 Optocoupler, U7 74AHC1G32, U8 LM555xM, U9 74AHC1G00

Commit message: BSPD + FL changes
Made BSPD and working on FL BOM
Parts:
- C10, C11, C15, C3, C4, C9: value 0.1u -> 100n
- C12: value 2.2u -> 1u; footprint Capacitor_SMD:C_0603_1608Metric -> Capacitor_SMD:C_0805_2012Metric
- C7: footprint Capacitor_SMD:C_0603_1608Metric -> Capacitor_SMD:C_0805_2012Metric
Routing:
- net GND: track 4.39 -> 0.17 mm, vias 128 -> 145

Commit message: Mostly Order ready BSPD and FL
Parts:
- removed the R4 at (108.3, 74.1)
- added R2: 1k, Resistor_SMD:R_0805_2012Metric, F.Cu at (103.4, 83.7)
- added R3: 10k, Resistor_SMD:R_0805_2012Metric, B.Cu at (108.2, 73.9)
- R12: renamed from R11; value 100k -> 225k
- moved C2 0.61 mm to (114.7, 74.7)
- moved C14 0.61 mm to (114.7, 99.7)
- moved C6 0.61 mm to (114.7, 87.3)
- moved R16 0.36 mm to (118.2, 87.3)
- moved R23 0.28 mm to (118.1, 99.8)
- moved C12 0.23 mm to (132.4, 108.1)
- moved C7 0.23 mm to (137.2, 101.7)
- renumbered R9 to R10, R10 to R11, R12 to R13, R13 to R14, R14 to R15, R15 to R16, R16 to R17, R17 to R18, R18 to R19, R19 to R20, R20 to R21, R21 to R22, R22 to R23, R23 to R24, R2 to R4, R3 to R5, R5 to R6, R6 to R7, R7 to R8, R8 to R9
Connections:
- U2 pad 3: Net-(U1-D) -> GND
- U2 pad 4: +5V -> Net-(U1-D)
Routing:
- net +5V: track 223.1 -> 232.4 mm, vias 15 -> 14
- net +12V: track 93.6 -> 99.7 mm, vias 6 -> 8
- net /Reset: track 70.8 -> 67.9 mm
- net /BMS_IN: track 9.88 -> 12.0 mm
- net Net-(U1-D): track 31.5 -> 31.7 mm, vias 3 -> 2
- net GND: vias 145 -> 174

Commit message: V1 of BSPD FL and Power ready for order
Parts:
- added R20: 0R, Resistor_SMD:R_0805_2012Metric, F.Cu at (115.2, 68.0)
- R12: value 225k -> 226k
- R5: value 1k -> 270R
- U10, U4: value SN74AHC1G08DBVR -> AND Gate
- U13, U3, U7: value 74AHC1G32 -> OR Gate
- U9: value 74AHC1G00 -> NAND Gate
- renumbered R20 to R21, R21 to R22, R22 to R23, R23 to R24, R24 to R25
Connections:
- J3 pad 06: +12V -> LVBat+
Routing:
- net +12V: track 99.7 -> 97.3 mm
- net LVBat+: track 0.00 -> 2.29 mm
- net GND: vias 174 -> 173
Other:
- board text added: "TR27 Fault Latch"
- board text removed: "FAULT LATCH TR27"
