File: Fault Latch 27/Fault Latch 27.kicad_pcb (KiCad board)
At the start: 2 copper layers, 37.6 x 50.9 mm, 97 parts, among them J1 Conn_01x01_Pin, J2 Conn_01x01_Pin, J3 Conn_01x06_Pin, J4 Conn_01x06_Pin, J5 Conn_01x01_Pin, K1 OJ-SS-112LMH2, K2 OJ-SS-112LMH2, K3 OJ-SS-112LMH2, Q1 Q_NMOS_GSD, Q10 Q_NMOS_GSD, Q11 Q_NMOS_GSD, Q2 Q_NMOS_GSD, Q3 Q_NMOS_GSD, Q4 Q_NMOS_GSD, Q5 Q_NMOS_GSD, Q6 Q_NMOS_GSD, Q7 Q_NMOS_GSD, Q8 Q_NMOS_GSD, Q9 Q_NMOS_GSD, SW1 SW_Omron_B3FS, U1 D-Latch, U10 AND Gate, U11 D-Latch, U12 Optocoupler, U13 OR Gate, U2 Optocoupler, U3 OR Gate, U4 AND Gate, U5 D-Latch, U6 Optocoupler, U7 OR Gate, U8 LM555xM, U9 NAND Gate

Commit message: fixed part # on bspd and fl
Connections:
- net LVBat+ renamed LV+
