File: Fault Latch 27/Fault Latch 27.kicad_sch (KiCad schematic)
At the start: 44 parts, among them K1 Relay_SPDT_Omron_G2RL-1, K2 Relay_SPDT_Omron_G2RL-1, K3 Relay_SPDT_Omron_G2RL-1, Q1 Q_NMOS_GSD, Q2 Q_NMOS_GSD, Q3 Q_NMOS_GSD, SW1 SW_Omron_B3FS, U1 74LVC1G373DBVRE4, U2 Optocoupler, U3 74AHC1G32, U4 74LVC1G373DBVRE4, U5 Optocoupler, U6 74AHC1G32, U7 74LVC1G373DBVRE4, U8 Optocoupler, U9 74AHC1G32

Commit message: FL27 finished schematic minus conectors
Parts:
- added C11: 1u, Capacitor_SMD:C_0603_1608Metric, symbol Device:C
- added C112, C113, C118: 0.1u, Capacitor_SMD:C_0402_1005Metric, symbol Device:C
- added C12: 100n, Capacitor_SMD:C_0603_1608Metric, symbol Device:C
- added C13: 2.2u, Capacitor_SMD:C_0603_1608Metric, symbol Device:C
- added Q105, Q106, Q112, Q113, Q114, Q115, Q4, Q5: Q_NMOS_GSD, Package_TO_SOT_SMD:SOT-23, symbol Transistor_FET:Q_NMOS_GSD
- added R112, R16, R18: 510R, Resistor_SMD:R_1210_3225Metric, symbol Device:R_US
- added R121, R136, R17: 10k, Resistor_SMD:R_1210_3225Metric, symbol Device:R_US
- added R130, R150: 270R, Resistor_SMD:R_1210_3225Metric, symbol Device:R_US
- added R133: 680R, Resistor_SMD:R_1210_3225Metric, symbol Device:R_US
- added R20: 100k, Resistor_SMD:R_1206_3216Metric, symbol Device:R_US
- added TP4: TestPoint, TestPoint:TestPoint_Pad_1.0x1.0mm, symbol Connector:TestPoint
- added U10: 74AHC1G00, symbol 74xGxx:74AHC1G00
- added U11, U12: SN74AHC1G08DBVR, Package_TO_SOT_SMD:SOT-23-5, symbol 74xGxx:74AHC1G08
- added U13: LM555xM, Package_SO:SOIC-8_3.9x4.9mm_P1.27mm, symbol Timer:LM555xM
- R2: value 2.2k -> 10k
- U1, U4, U7: value 74LVC1G373DBVRE4 -> D-Latch
Connections:
- net +12V: now also R121.1, R136.1, R17.1
- net +5V: now also C11.1, C112.2, C113.2, C118.2, C12.1, U10.5 (VCC), U11.5 (VCC), U12.5 (VCC), U13.4 (R), U13.8 (VCC)
- net GND: now also C11.2, C112.1, C113.1, C118.1, C12.2, C13.2, Q105.2 (S), Q106.2 (S), Q112.2 (S), Q113.2 (S), Q114.2 (S), Q115.2 (S), Q4.2 (S), Q5.2 (S), U10.3 (GND), U11.3 (GND), U12.3 (GND), U13.1 (GND)
- net BMS LE renamed BMS_LE
- net BMS Q renamed BMS_Q
- net BMS_Q: now also Q114.1 (G), U10.2, U12.1
- net BSPD IN renamed BSPD_IN
- net BSPD LE renamed BSPD_LE
- net BSPD Q renamed BSPD_Q
- net BSPD_Q: now also Q4.1 (G)
- net IMD IN renamed IMD_IN
- net IMD LE renamed IMD_LE
- net IMD Q renamed IMD_Q
- net IMD_Q: now also Q105.1 (G), U10.1, U12.2
- net Shutdown IN renamed Shutdown_IN
- net Shutdown OUT renamed Shutdown_OUT
- new net: U10.4, U11.1
- new net: R133.2, U11.4
- new net: Q105.3 (D), Q106.1 (G), R121.2
- new net: Q4.3 (D), Q5.1 (G), R17.2
- new net: Q106.3 (D), R112.2
- new net: Q114.3 (D), Q115.1 (G), R136.2
- new net: Q5.3 (D), R18.2
- new net: Q112.1 (G), U12.4
- new net: Q112.3 (D), R130.1
- new net: Q115.3 (D), R16.2
- new net: Q113.1 (G), R133.1
- new net: Q113.3 (D), R150.1
- new net BMS Light -: R16.1
- new net BSPD Light -: R18.1
- new net CLOCK: R20.2, TP4.1, U11.2, U13.3 (Q)
- new net IMD Light -: R112.1
- new net THRESH: C13.1, R20.1, U13.2 (TR), U13.6 (THR)
- new net TSSI Green -: R130.2
- new net TSSI Red -: R150.2
- no-connect marks 0 -> 2
Other:
- note added: "3-5hz 50% Clock"
- note added: "BMS Fault Light"
- note added: "BMS_LE"
- note added: "BSPD Fault Light"
- note added: "BSPD_LE"
- note added: "IMD Fault Light"
- note added: "IMD_LE"
- note added: "Reset Button"
- note added: "TSSI Green"
- note added: "TSSI Red"
- note added: "falstad: https://tinyurl.com/29v9662o"
- moved on the sheet: C2, SW1

Commit message: V1 FL27 Done
Need to double check components for everything + footprints
Parts:
- removed K1, K2, K3: Relay_SPDT_Omron_G2RL-1, Relay_THT:Relay_SPDT_Omron_G2RL-1, symbol Relay:G2RL-1
- removed R112, R16, R18: 510R, Resistor_SMD:R_1210_3225Metric, symbol Device:R_US
- removed R130, R150: 270R, Resistor_SMD:R_1210_3225Metric, symbol Device:R_US
- removed U5, U8: Optocoupler, symbol Isolator:Optocoupler_DC_PhotoNPN_AKEC
- added C1, C13, C5: 100n, Capacitor_SMD:C_0603_1608Metric, symbol Device:C
- added D1, D4, D7: (no value), Diode_SMD:D_SOD-323, symbol Diode:1N914
- added H1, H2, H3, H4: MountingHole, MountingHole:MountingHole_3.2mm_M3_DIN965_Pad, symbol Mechanical:MountingHole
- added J1, J2, J5: Conn_01x01_Pin, 1.Custom_Footprints:SAMTEC_TSW-101-07-L-S, symbol Connector:Conn_01x01_Pin
- added J3, J4: Conn_01x06_Pin, 1.Custom_Footprints:SAMTEC_TSW-103-07-L-D, symbol Connector:Conn_01x06_Pin
- added K1, K2, K3: OJ-SS-112LMH2, 1.Custom_Footprints:OJSS112LMH2, symbol Relay:Fujitsu_FTR-LYAA005x
- added R14, R21, R4: 10k, Resistor_SMD:R_0805_2012Metric, symbol Device:R_US
- added TP1, TP2, TP3, TP4, TP6, TP7: TestPoint, TestPoint:TestPoint_Pad_1.0x1.0mm, symbol Connector:TestPoint
- added U12, U6: Optocoupler, 1.Custom_Footprints:SSOP-4_VOS617A_VIS, symbol Isolator:Optocoupler_DC_PhotoNPN_AKEC
- C10: renamed from C112; footprint Capacitor_SMD:C_0402_1005Metric -> Capacitor_SMD:C_0603_1608Metric
- C11: renamed from C113; footprint Capacitor_SMD:C_0402_1005Metric -> Capacitor_SMD:C_0603_1608Metric
- C14: renamed from C6; footprint Capacitor_SMD:C_0603_1608Metric_Pad1.08x0.95mm_HandSolder -> Capacitor_SMD:C_0603_1608Metric
- C15: renamed from C7; footprint Capacitor_SMD:C_0402_1005Metric -> Capacitor_SMD:C_0603_1608Metric
- C16: renamed from C2; footprint Capacitor_SMD:C_0603_1608Metric_Pad1.08x0.95mm_HandSolder -> Capacitor_SMD:C_0603_1608Metric
- C2: renamed from C1; footprint Capacitor_SMD:C_0603_1608Metric_Pad1.08x0.95mm_HandSolder -> Capacitor_SMD:C_0603_1608Metric
- C3: footprint Capacitor_SMD:C_0402_1005Metric -> Capacitor_SMD:C_0603_1608Metric
- C4: renamed from C118; footprint Capacitor_SMD:C_0402_1005Metric -> Capacitor_SMD:C_0603_1608Metric
- C6: renamed from C4; footprint Capacitor_SMD:C_0603_1608Metric_Pad1.08x0.95mm_HandSolder -> Capacitor_SMD:C_0603_1608Metric
- C9: renamed from C5; footprint Capacitor_SMD:C_0402_1005Metric -> Capacitor_SMD:C_0603_1608Metric
- R1, R2, R3: footprint Resistor_SMD:R_1210_3225Metric -> Resistor_SMD:R_0805_2012Metric
- R10: renamed from R6; footprint Resistor_SMD:R_1210_3225Metric -> Resistor_SMD:R_0805_2012Metric
- R11: renamed from R20; footprint Resistor_SMD:R_1206_3216Metric -> Resistor_SMD:R_0805_2012Metric
- R12: renamed from R7; footprint Resistor_SMD:R_1210_3225Metric -> Resistor_SMD:R_1206_3216Metric
- R13: renamed from R8; footprint Resistor_SMD:R_1210_3225Metric -> Resistor_SMD:R_0805_2012Metric
- R15: renamed from R9; footprint Resistor_SMD:R_1210_3225Metric -> Resistor_SMD:R_0805_2012Metric
- R16: renamed from R10; value 100k -> 10k; footprint Resistor_SMD:R_1210_3225Metric -> Resistor_SMD:R_0805_2012Metric
- R17: renamed from R133; footprint Resistor_SMD:R_1210_3225Metric -> Resistor_SMD:R_0805_2012Metric
- R18: renamed from R11; footprint Resistor_SMD:R_1210_3225Metric -> Resistor_SMD:R_0805_2012Metric
- R19: renamed from R12; footprint Resistor_SMD:R_1210_3225Metric -> Resistor_SMD:R_0805_2012Metric
- R20: renamed from R13; footprint Resistor_SMD:R_1210_3225Metric -> Resistor_SMD:R_0805_2012Metric
- R22: renamed from R14; footprint Resistor_SMD:R_1210_3225Metric -> Resistor_SMD:R_0805_2012Metric
- R23: renamed from R15; value 100k -> 10k; footprint Resistor_SMD:R_1210_3225Metric -> Resistor_SMD:R_0805_2012Metric
- R5: renamed from R4; footprint Resistor_SMD:R_1210_3225Metric -> Resistor_SMD:R_0805_2012Metric
- R6: renamed from R5; value 100k -> 10k; footprint Resistor_SMD:R_1210_3225Metric -> Resistor_SMD:R_0805_2012Metric
- R7: renamed from R121; footprint Resistor_SMD:R_1210_3225Metric -> Resistor_SMD:R_0805_2012Metric
- R8: renamed from R136; footprint Resistor_SMD:R_1210_3225Metric -> Resistor_SMD:R_0805_2012Metric
- R9: renamed from R17; footprint Resistor_SMD:R_1210_3225Metric -> Resistor_SMD:R_0805_2012Metric
- U1: footprint Package_TO_SOT_SMD:SOT-23-6 -> Package_TO_SOT_SMD:SOT-363_SC-70-6
- U10: renamed from U11; footprint Package_TO_SOT_SMD:SOT-23-5 -> Package_TO_SOT_SMD:SOT-353_SC-70-5
- U11: renamed from U7; footprint Package_TO_SOT_SMD:SOT-23-6 -> Package_TO_SOT_SMD:SOT-363_SC-70-6
- U13: renamed from U9; footprint (none) -> Package_TO_SOT_SMD:SOT-353_SC-70-5
- U2: footprint (none) -> 1.Custom_Footprints:SSOP-4_VOS617A_VIS; MF# (none) -> VOS617A-3T
- U3: footprint (none) -> Package_TO_SOT_SMD:SOT-353_SC-70-5
- U4: renamed from U12; footprint Package_TO_SOT_SMD:SOT-23-5 -> Package_TO_SOT_SMD:SOT-353_SC-70-5
- U5: renamed from U4; footprint Package_TO_SOT_SMD:SOT-23-6 -> Package_TO_SOT_SMD:SOT-363_SC-70-6
- U7: renamed from U6; footprint (none) -> Package_TO_SOT_SMD:SOT-353_SC-70-5
- U9: renamed from U10; footprint (none) -> Package_TO_SOT_SMD:SOT-353_SC-70-5
- renumbered C13 to C12, C11 to C7, C12 to C8, D1 to D2, D2 to D3, D3 to D5, D4 to D6, D5 to D8, D6 to D9, Q113 to Q10, Q3 to Q11, Q106 to Q2, Q115 to Q3, Q5 to Q4, Q112 to Q5, Q105 to Q6, Q114 to Q7, Q4 to Q8, Q2 to Q9, TP4 to TP5, U13 to U8
Connections:
- net +12V: now also D1.1 (K), D4.1 (K), D7.1 (K), J3.06 (Pin_6), K1.2, K2.2, K3.2
- net +5V: now also C1.1, C13.1, C5.1, J4.06 (Pin_6), U12.4, U6.4
- net BMS Light -: now also Q3.3 (D), J3.04 (Pin_4)
- net BMS_Q: now also TP2.1
- net BSPD Light -: now also Q4.3 (D), J4.03 (Pin_3)
- net BSPD_IN: now also J5.01 (Pin_1), U12.1; no longer C3.1, D3.2 (A2), R2.2, U2.1
- net BSPD_Q: now also TP7.1
- net GND: now also C1.2, C13.2, C5.2, J3.01 (Pin_1), J4.01 (Pin_1), R14.1, R21.1, R4.1
- net IMD Light -: now also Q2.3 (D), J4.05 (Pin_5)
- net IMD_IN: now also J2.01 (Pin_1), U6.1
- net IMD_Q: now also TP4.1
- net Reset: now also J3.05 (Pin_5)
- net Shutdown_IN: now also J3.03 (Pin_3), K1.4
- net Shutdown_OUT: now also J4.04 (Pin_4), K3.3
- net TSSI Green -: now also Q5.3 (D), J3.02 (Pin_2)
- net TSSI Red -: now also Q10.3 (D), J4.02 (Pin_2)
- net at Q1.3 (D): now also D1.2 (A), K1.1
- net at C15.2, R20.2: now also U12.2
- net at Q9.3 (D): now also D4.2 (A), K2.1
- net at C9.2, R13.2: now also U6.2
- net at Q11.3 (D): now also D7.2 (A), K3.1
- net at U5.3 (D): now also R14.2, TP3.1, U6.3
- net at U11.3 (D): now also R21.2, TP6.1, U12.3
- net at U1.3 (D), U2.3: now also R4.2, TP1.1
- new net: K2.3, K3.4
- new net: K1.3, K2.4
- new net BMS_IN: C3.1, D3.2 (A2), J1.01 (Pin_1), R2.2, U2.1
Other:
- moved on the sheet: Q5, R1, R10, R18

Commit message: BSPD + FL changes
Made BSPD and working on FL BOM
Parts:
- C1, C13, C14, C16, C2, C5, C6, C8: $/unit Digikey (none) -> $0.19; $/unit Mouser (none) -> $0.15; Digikey# (none) -> 311-3034-2-ND; MF# (none) -> AC0603KRX7R9BB104; Mouser# (none) -> 603-AC0603KR9BB104
- C10, C11, C15, C3, C4, C9: value 0.1u -> 100n; $/unit Digikey (none) -> $0.19; $/unit Mouser (none) -> $0.15; Digikey# (none) -> 311-3034-2-ND; MF# (none) -> AC0603KRX7R9BB104; Mouser# (none) -> 603-AC0603KR9BB104
- C12: value 2.2u -> 1u; footprint Capacitor_SMD:C_0603_1608Metric -> Capacitor_SMD:C_0805_2012Metric; $/unit Digikey (none) -> $0.59; $/unit Mouser (none) -> $0.49; Digikey# (none) -> 13-AC0805KKX7R9BB105TR-ND; MF# (none) -> AC0805KKX7R9BB105; Mouser# (none) -> 603-AC0805KKX7R9B105
- C7: footprint Capacitor_SMD:C_0603_1608Metric -> Capacitor_SMD:C_0805_2012Metric; $/unit Digikey (none) -> $0.59; $/unit Mouser (none) -> $0.49; Digikey# (none) -> 13-AC0805KKX7R9BB105TR-ND; MF# (none) -> AC0805KKX7R9BB105; Mouser# (none) -> 603-AC0805KKX7R9B105
- D1, D4, D7: $/unit Digikey (none) -> $0.11; $/unit Mouser (none) -> N/A; Digikey# (none) -> 5399-1N4007WSTR-ND; MF# (none) -> 1N4007WS; Mouser# (none) -> N/A
- D2, D5, D8: $/unit Digikey (none) -> $0.17; $/unit Mouser (none) -> $0.29; Digikey# (none) -> 475-LSR976-NR-1TR-ND; JLC# C19171391 -> (none); MF# (none) -> Q62702P5178; Mouser# (none) -> 720-Q62702P5178
- D3, D6, D9: $/unit Digikey (none) -> $0.73; $/unit Mouser (none) -> $0.69; Digikey# (none) -> 641-2082-2-ND; MF# (none) -> CPDUR12V-HF
- K1, K2, K3: $/unit Digikey (none) -> $2.50; $/unit Mouser (none) -> $2.50; Digikey# (none) -> PB1981-ND; MF# (none) -> OJ-SS-112LMH2; Mouser# (none) -> 655-OJ-SS-112LMH2
- Q1, Q10, Q11, Q2, Q3, Q4, Q5, Q6, Q7, Q8, Q9: $/unit Digikey (none) -> $0.16; $/unit Mouser (none) -> $0.15; Digikey# (none) -> 4878-MMFTN6001TR-ND; MF# (none) -> MMFTN6001; Mouser# (none) -> 637-MMFTN6001
- R11: value 100k -> 225k
- U12, U2, U6: $/unit Digikey (none) -> $0.57; $/unit Mouser (none) -> $0.56; Digikey# (none) -> VOS617A-3TTR-ND; Mouser# (none) -> 78-VOS617A-3T

Commit message: Mostly Order ready BSPD and FL
Parts:
- removed R4: 10k, Resistor_SMD:R_0805_2012Metric, symbol Device:R_US
- added R2: 1k, Resistor_SMD:R_0805_2012Metric, symbol Device:R_US
- added R3: 10k, Resistor_SMD:R_0805_2012Metric, symbol Device:R_US
- C12, C7: Digikey# 13-AC0805KKX7R9BB105TR-ND -> 13-AC0805KKX7R9BB105CT-ND
- D1, D4, D7: Digikey# 5399-1N4007WSTR-ND -> 5399-1N4007WSCT-ND
- D2, D5, D8: Digikey# 475-LSR976-NR-1TR-ND -> 475-LSR976-NR-1CT-ND
- Q1, Q10, Q11, Q2, Q3, Q4, Q5, Q6, Q7, Q8, Q9: Digikey# 4878-MMFTN6001TR-ND -> 4878-MMFTN6001CT-ND
- R1: $/unit Digikey (none) -> $0.10; $/unit Mouser (none) -> $0.10; Digikey# (none) -> 311-2.00KCRCT-ND; MF# (none) -> RC0805FR-072KL; Mouser# (none) -> 603-RC0805FR-072KL
- R10: renamed from R9; $/unit Digikey (none) -> $0.10; $/unit Mouser (none) -> $0.10; Digikey# (none) -> 311-10.0KCRCT-ND; MF# (none) -> RC0805FR-0710KL; Mouser# (none) -> 603-RC0805FR-0710KL
- R11: renamed from R10; $/unit Digikey (none) -> $0.10; $/unit Mouser (none) -> $0.10; Digikey# (none) -> 311-2.00KCRCT-ND; MF# (none) -> RC0805FR-072KL; Mouser# (none) -> 603-RC0805FR-072KL
- R12: renamed from R11; value 225k -> 226k; $/unit Digikey (none) -> $0.10; $/unit Mouser (none) -> $0.10; Digikey# (none) -> 311-226KCRCT-ND; MF# (none) -> RC0805FR-07226KL; Mouser# (none) -> 603-RC0805FR-07226KL
- R13: renamed from R12; $/unit Digikey (none) -> $0.17; $/unit Mouser (none) -> $0.17; Digikey# (none) -> 2019-SG73P2BTTD2201FCT-ND; MF# (none) -> SG73P2BTTD2201F; Mouser# (none) -> 660-SG73P2BTTD2201F
- R14: renamed from R13; $/unit Digikey (none) -> $0.10; $/unit Mouser (none) -> $0.10; Digikey# (none) -> 311-1.00KCRCT-ND; MF# (none) -> RC0805FR-071KL; Mouser# (none) -> 603-RC0805FR-071KL
- R15: renamed from R14; $/unit Digikey (none) -> $0.10; $/unit Mouser (none) -> $0.10; Digikey# (none) -> 311-10.0KCRCT-ND; MF# (none) -> RC0805FR-0710KL; Mouser# (none) -> 603-RC0805FR-0710KL
- R16: renamed from R15; $/unit Digikey (none) -> $0.10; $/unit Mouser (none) -> $0.10; Digikey# (none) -> 311-10.0KCRCT-ND; MF# (none) -> RC0805FR-0710KL; Mouser# (none) -> 603-RC0805FR-0710KL
- R17: renamed from R16; $/unit Digikey (none) -> $0.10; $/unit Mouser (none) -> $0.10; Digikey# (none) -> 311-10.0KCRCT-ND; MF# (none) -> RC0805FR-0710KL; Mouser# (none) -> 603-RC0805FR-0710KL
- R18: renamed from R17; $/unit Digikey (none) -> $0.10; $/unit Mouser (none) -> $0.10; Digikey# (none) -> 311-680CRCT-ND; MF# (none) -> RC0805FR-07680RL; Mouser# (none) -> 603-RC0805FR-07680RL
- R19: renamed from R18; $/unit Digikey (none) -> $0.10; $/unit Mouser (none) -> $0.10; Digikey# (none) -> 311-2.00KCRCT-ND; MF# (none) -> RC0805FR-072KL; Mouser# (none) -> 603-RC0805FR-072KL
- R20: renamed from R19; $/unit Digikey (none) -> $0.10; $/unit Mouser (none) -> $0.10; Digikey# (none) -> 311-10.0KCRCT-ND; MF# (none) -> RC0805FR-0710KL; Mouser# (none) -> 603-RC0805FR-0710KL
- R21: renamed from R20; $/unit Digikey (none) -> $0.10; $/unit Mouser (none) -> $0.10; Digikey# (none) -> 311-1.00KCRCT-ND; MF# (none) -> RC0805FR-071KL; Mouser# (none) -> 603-RC0805FR-071KL
- R22: renamed from R21; $/unit Digikey (none) -> $0.10; $/unit Mouser (none) -> $0.10; Digikey# (none) -> 311-10.0KCRCT-ND; MF# (none) -> RC0805FR-0710KL; Mouser# (none) -> 603-RC0805FR-0710KL
- R23: renamed from R22; $/unit Digikey (none) -> $0.10; $/unit Mouser (none) -> $0.10; Digikey# (none) -> 311-10.0KCRCT-ND; MF# (none) -> RC0805FR-0710KL; Mouser# (none) -> 603-RC0805FR-0710KL
- R24: renamed from R23; $/unit Digikey (none) -> $0.10; $/unit Mouser (none) -> $0.10; Digikey# (none) -> 311-10.0KCRCT-ND; MF# (none) -> RC0805FR-0710KL; Mouser# (none) -> 603-RC0805FR-0710KL
- R4: renamed from R2; $/unit Digikey (none) -> $0.10; $/unit Mouser (none) -> $0.10; Digikey# (none) -> 311-10.0KCRCT-ND; MF# (none) -> RC0805FR-0710KL; Mouser# (none) -> 603-RC0805FR-0710KL
- R5: renamed from R3; $/unit Digikey (none) -> $0.10; $/unit Mouser (none) -> $0.10; Digikey# (none) -> 311-1.00KCRCT-ND; MF# (none) -> RC0805FR-071KL; Mouser# (none) -> 603-RC0805FR-071KL
- R6: renamed from R5; $/unit Digikey (none) -> $0.10; $/unit Mouser (none) -> $0.10; Digikey# (none) -> 311-10.0KCRCT-ND; MF# (none) -> RC0805FR-0710KL; Mouser# (none) -> 603-RC0805FR-0710KL
- R7: renamed from R6; $/unit Digikey (none) -> $0.10; $/unit Mouser (none) -> $0.10; Digikey# (none) -> 311-10.0KCRCT-ND; MF# (none) -> RC0805FR-0710KL; Mouser# (none) -> 603-RC0805FR-0710KL
- R8: renamed from R7; $/unit Digikey (none) -> $0.10; $/unit Mouser (none) -> $0.10; Digikey# (none) -> 311-10.0KCRCT-ND; MF# (none) -> RC0805FR-0710KL; Mouser# (none) -> 603-RC0805FR-0710KL
- R9: renamed from R8; $/unit Digikey (none) -> $0.10; $/unit Mouser (none) -> $0.10; Digikey# (none) -> 311-10.0KCRCT-ND; MF# (none) -> RC0805FR-0710KL; Mouser# (none) -> 603-RC0805FR-0710KL
- SW1: $/unit Digikey (none) -> $0.75; $/unit Mouser (none) -> $0.73; Digikey# (none) -> SW423CT-ND; MF# (none) -> B3FS-1000P; Mouser# (none) -> 653-B3FS-1000P
- TP1, TP2, TP3, TP4, TP5, TP6, TP7: now left out of the parts list
- U1, U11, U5: $/unit Digikey (none) -> $0.28; $/unit Mouser (none) -> $0.28; Digikey# (none) -> 296-18775-1-ND; MF# (none) -> SN74LVC1G373DCKR; Mouser# (none) -> 595-SN74LVC1G373DCKR
- U10, U4: value SN74AHC1G08DBVR -> AND Gate; $/unit Digikey (none) -> $0.19; $/unit Mouser (none) -> $0.19; Digikey# (none) -> 296-18066-1-ND; MF# (none) -> SN74LVC1G11DCKR; Mouser# (none) -> 595-SN74LVC1G11DCKR
- U13, U3, U7: value 74AHC1G32 -> OR Gate; $/unit Digikey (none) -> $0.11; $/unit Mouser (none) -> $0.11; Digikey# (none) -> 296-9848-1-ND; MF# (none) -> SN74LVC1G32DCKR; Mouser# (none) -> 595-SN74LVC1G32DCKR
- U8: $/unit Digikey (none) -> $1.15; $/unit Mouser (none) -> $1.15; Digikey# (none) -> LMC555CMX/NOPBCT-ND; MF# (none) -> LMC555CMX/NOPB; Mouser# (none) -> 926-LMC555CMX/NOPB
- U9: value 74AHC1G00 -> NAND Gate; $/unit Digikey (none) -> $0.11; $/unit Mouser (none) -> $0.11; Digikey# (none) -> 296-9846-1-ND; MF# (none) -> SN74LVC1G00DCKR; Mouser# (none) -> 595-SN74LVC1G00DCKR
Connections:
- net +12V: now also R2.2
- net +5V: now also R3.1; no longer U2.4
- net BMS_IN: now also R2.1
- net GND: now also U2.3
- net at TP1.1, U1.3 (D): now also U2.4, R3.2; no longer U2.3

Commit message: V1 of BSPD FL and Power ready for order
Parts:
- added R20: 0R, Resistor_SMD:R_0805_2012Metric, symbol Device:R_US
- R5: value 1k -> 270R; $/unit Digikey $0.10 -> (none); $/unit Mouser $0.10 -> (none); Digikey# 311-1.00KCRCT-ND -> (none); JLC# C137088 -> (none); MF# RC0805FR-071KL -> (none); MOUSER 603-RC1210JR-0710KL -> (none); Mouser# 603-RC0805FR-071KL -> (none)
- renumbered R20 to R21, R21 to R22, R22 to R23, R23 to R24, R24 to R25
Connections:
- net +12V: now also R20.1; no longer J3.06 (Pin_6)
- new net LV+: J3.06 (Pin_6), R20.2
