File: Fault Latch 27/Fault Latch 27.kicad_sch (KiCad schematic)
At the start: 94 parts, among them J1 Conn_01x01_Pin, J2 Conn_01x01_Pin, J3 Conn_01x06_Pin, J4 Conn_01x06_Pin, J5 Conn_01x01_Pin, K1 OJ-SS-112LMH2, K2 OJ-SS-112LMH2, K3 OJ-SS-112LMH2, Q1 Q_NMOS_GSD, Q10 Q_NMOS_GSD, Q11 Q_NMOS_GSD, Q2 Q_NMOS_GSD, Q3 Q_NMOS_GSD, Q4 Q_NMOS_GSD, Q5 Q_NMOS_GSD, Q6 Q_NMOS_GSD, Q7 Q_NMOS_GSD, Q8 Q_NMOS_GSD, Q9 Q_NMOS_GSD, SW1 SW_Omron_B3FS, U1 D-Latch, U10 AND Gate, U11 D-Latch, U12 Optocoupler, U13 OR Gate, U2 Optocoupler, U3 OR Gate, U4 AND Gate, U5 D-Latch, U6 Optocoupler, U7 OR Gate, U8 LM555xM, U9 NAND Gate

Commit message: fixed part # on bspd and fl
Parts:
- C1, C10, C11, C13, C14, C15, C16, C2, C3, C4, C5, C6, C8, C9: Digikey# 311-3034-2-ND -> (none)
- C12, C7: Digikey# 13-AC0805KKX7R9BB105CT-ND -> (none)
- D2, D5, D8: Mouser# 720-Q62702P5178 -> (none)
- D3, D6, D9: Digikey# 641-2082-2-ND -> (none)
- K1, K2, K3: Digikey# PB1981-ND -> (none)
- Q1, Q10, Q11, Q2, Q3, Q4, Q5, Q6, Q7, Q8, Q9: Digikey# 4878-MMFTN6001CT-ND -> (none)
- R1, R11, R19: Digikey# 311-2.00KCRCT-ND -> (none)
- R10, R15, R16, R17, R21, R23, R24, R25, R3, R4, R6, R7, R8, R9: Mouser# 603-RC0805FR-0710KL -> (none)
- R12: Digikey# 311-226KCRCT-ND -> (none)
- R13: Digikey# 2019-SG73P2BTTD2201FCT-ND -> (none)
- R14, R2, R22: Mouser# 603-RC0805FR-071KL -> (none)
- R18: Digikey# 311-680CRCT-ND -> (none)
- SW1: Digikey# SW423CT-ND -> (none)
- U1, U11, U5: Mouser# 595-SN74LVC1G373DCKR -> (none)
- U10, U4: Digikey# 296-18066-1-ND -> (none)
- U12, U2, U6: Mouser# 78-VOS617A-3T -> (none)
- U13, U3, U7: Digikey# 296-9848-1-ND -> (none)
- U8: Digikey# LMC555CMX/NOPBCT-ND -> (none)
- U9: Digikey# 296-9846-1-ND -> (none)
