File: Precharge 27/Precharge 27.kicad_sch (KiCad schematic)
At the start: 0 parts

Commit message: fixed footprints and mouser# for rml
Other:
- note added: "PRECHARGE 27"
Changed lines of the file:
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@@
 	(generator_version "10.0")
 	(paper "A4")
+	(text "PRECHARGE 27\n"
+		(exclude_from_sim no)
+		(at 27.432 15.494 0)
+		(effects
+			(font
+				(size 2.54 2.54)
+				(thickness 0.508)
+				(bold yes)
+			)
+		)
+	)
 	(sheet_instances
 		(path "/"
