File: Module Lids/Module Lids.kicad_pcb (KiCad board)
At the start: 2 copper layers, 50.8 x 483.6 mm, 9 parts

Commit message: added module lids and fixed RML part #s
Parts:
- removed J**: 2068321401, Module Lids:14-Pin-Molex
- removed J** (x4): SHDRRA8W50P0X200_1X8_1790X760X480P, Module Lids:8-Pin-JST
- removed J**: B24BPADSS1FLFSN, Module Lids:24-Pin-JST
- removed J** (x3): 215760-YY05, Module Lids:5-Pin-Molex
- added CT1: Celltap 1, Module Lids:5-Pin-Molex, B.Cu at (538.0, 449.1)
- added CT2: Celltap 1, Module Lids:5-Pin-Molex, B.Cu at (538.0, 305.3)
- added CT3: Celltap 1, Module Lids:5-Pin-Molex, B.Cu at (549.9, 272.6)
- added CT4: Celltap Conn, Module Lids:14-Pin-Molex, F.Cu at (553.0, 138.2)
- added F1: Fuse_Small, Fuse:Fuse_1206_3216Metric_Pad1.42x1.75mm_HandSolder, B.Cu at (538.0, 444.3)
- added F10: Fuse_Small, Fuse:Fuse_1206_3216Metric_Pad1.42x1.75mm_HandSolder, B.Cu at (546.9, 277.3)
- added F11: Fuse_Small, Fuse:Fuse_1206_3216Metric_Pad1.42x1.75mm_HandSolder, B.Cu at (543.9, 277.3)
- added F12: Fuse_Small, Fuse:Fuse_1206_3216Metric_Pad1.42x1.75mm_HandSolder, B.Cu at (540.9, 277.3)
- added F13: Fuse_Small, Fuse:Fuse_1206_3216Metric_Pad1.42x1.75mm_HandSolder, B.Cu at (550.0, 444.3)
- added F2: Fuse_Small, Fuse:Fuse_1206_3216Metric_Pad1.42x1.75mm_HandSolder, B.Cu at (541.0, 444.3)
- added F3: Fuse_Small, Fuse:Fuse_1206_3216Metric_Pad1.42x1.75mm_HandSolder, B.Cu at (544.0, 444.3)
- added F4: Fuse_Small, Fuse:Fuse_1206_3216Metric_Pad1.42x1.75mm_HandSolder, B.Cu at (547.0, 444.3)
- added F5: Fuse_Small, Fuse:Fuse_1206_3216Metric_Pad1.42x1.75mm_HandSolder, B.Cu at (538.0, 300.6)
- added F6: Fuse_Small, Fuse:Fuse_1206_3216Metric_Pad1.42x1.75mm_HandSolder, B.Cu at (541.0, 300.6)
- added F7: Fuse_Small, Fuse:Fuse_1206_3216Metric_Pad1.42x1.75mm_HandSolder, B.Cu at (544.0, 300.6)
- added F8: Fuse_Small, Fuse:Fuse_1206_3216Metric_Pad1.42x1.75mm_HandSolder, B.Cu at (547.0, 300.6)
- added F9: Fuse_Small, Fuse:Fuse_1206_3216Metric_Pad1.42x1.75mm_HandSolder, B.Cu at (549.9, 277.3)
- added J1: B24B-PADSS-1F_LF__SN_, Module Lids:24-Pin-JST, F.Cu at (512.2, 142.7)
- added J2: S10B-PADSS-1_LF__SN_, Module Lids:10-Pin-JST, F.Cu at (506.2, 213.0)
- added J3: S10B-PADSS-1_LF__SN_, Module Lids:10-Pin-JST, F.Cu at (506.5, 373.0)
- added J4: S10B-PADSS-1_LF__SN_, Module Lids:10-Pin-JST, F.Cu at (505.2, 535.5)
Routing:
- net /T_1: track 0.00 -> 441.2 mm
- net /T_2: track 0.00 -> 435.0 mm
- net /T_3: track 0.00 -> 432.1 mm
- net /T_4: track 0.00 -> 429.1 mm
- net /T_GND: track 0.00 -> 427.3 mm
- net /T_6: track 0.00 -> 426.5 mm
- net /T_5: track 0.00 -> 426.3 mm
- net Net-(CT4-Pad4): track 0.00 -> 358.8 mm
- net Net-(CT4-Pad2): track 0.00 -> 356.9 mm
- net Net-(CT4-Pad3): track 0.00 -> 341.2 mm, vias 0 -> 1
- net Net-(CT4-Pad1): track 0.00 -> 339.6 mm, vias 0 -> 1
- net Net-(CT4-Pad13): track 0.00 -> 326.6 mm, vias 0 -> 1
- net /T_7: track 0.00 -> 253.1 mm
- net /T_8: track 0.00 -> 248.2 mm
- net /T_12: track 0.00 -> 245.1 mm
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Other:
- board size 50.8 x 483.6 mm -> 57.8 x 451.5 mm
- board text added: "BMS Side"
- board text added: "JLC +- 0.2mm tolerance"
- board text added: "Plug Side"
