File: RML Constant Current/RML_EMO/RML_EMO.kicad_sch (KiCad schematic)
At the start: 49 parts, among them J1 Tyco, J2 NANOFIT-4PIN, J3 Tyco, Q3 Q_NMOS_GSD, Q4 Q_NMOS_GSD, Q5 Q_NMOS_GSD, U1 LR8K4-G, U2 LM555xM, U5 LM1117DT-5.0, U6 Optocoupler, U7 74AHC1G02, U8 OPA1662DGK

Commit message: Current sink resistor change and DRC fix
Parts:
- R12: value 1.8k -> 6k
Changed lines of the file:
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@@
 			)
 		)
-		(property "Value" "1.8k"
+		(property "Value" "6k"
 			(at 138.43 90.678 90)
 			(show_name no)

Commit message: added mouser# to HV side components
Parts:
- removed TP4: TestPoint, TestPoint:TestPoint_Pad_1.0x1.0mm, symbol Connector:TestPoint
- C11: JLC# (none) -> C1592
- C4, C7: JLC# (none) -> C91186
- D1: footprint Diode_SMD:D_TUMD2 -> Diode_SMD:D_SOD-523; Mouser# (none) -> 755-RFU01SM4ST2R
- Q5: Digikey# (none) -> IPP60R180P7XKSA1-ND
- R1: Mouser# (none) -> 603-RC0805FR-10100KL
- R10: value 97.5k -> 86.6k; Mouser# (none) -> 667-ERJ-P06F8662V
- R11: Mouser# (none) -> 667-ERJ-P06J105V
- R12: value 6k -> 6.04k; Mouser# (none) -> 667-ERJ-P06F6041V
- R2: Mouser# (none) -> 652-CR0805FX-3571ELF
- R3: value 400K -> 374k; footprint Resistor_SMD:R_0805_2012Metric_Pad1.20x1.40mm_HandSolder -> Resistor_SMD:R_0805_2012Metric; Mouser# (none) -> 71-CRCW0805400KJNTA
- R4: value 37K -> 36k; Mouser# (none) -> 667-ERJ-P06F3602V
- R7: value 85.6k -> 86.6k; Mouser# (none) -> 667-ERJ-P06F8662V
- R8: value 14.4k -> 14.3k; Mouser# (none) -> 667-ERJ-P06F1432V
- R9: value 2.5k -> 2k; Mouser# (none) -> 71-CRCW08052K00JNEA
Connections:
- net 5.17V renamed 5.10V

Commit message: added bleeder resistor
Parts:
- added R17: 1.5M, Resistor_SMD:R_2010_5025Metric_Pad1.40x2.65mm_HandSolder, symbol Device:R_US
- C2: Mouser# (none) -> 810-CAA572X6T2W225M6
Connections:
- net GNDPWR: now also R17.1
- net HVI+: now also R17.2
Other:
- moved on the sheet: C2
Changed lines of the file:
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@@
 	)
 	(junction
+		(at 26.67 22.86)
+		(diameter 0)
+		(color 0 0 0 0)
+	)
+	(junction
 		(at 127 110.49)
 		(diameter 0)
@@
 	)
 	(junction
-		(at 30.48 22.86)
+		(at 168.91 26.67)
 		(diameter 0)
 		(color 0 0 0 0)
 	)
 	(junction
-		(at 168.91 26.67)
+		(at 48.26 34.29)
 		(diameter 0)
 		(color 0 0 0 0)
 	)
 	(junction
-		(at 48.26 34.29)
+		(at 29.21 156.21)
 		(diameter 0)
 		(color 0 0 0 0)
 	)
 	(junction
-		(at 29.21 156.21)
+		(at 33.02 22.86)
 		(diameter 0)
 		(color 0 0 0 0)
@@
 	)
 	(junction
+		(at 26.67 33.02)
+		(diameter 0)
+		(color 0 0 0 0)
+	)
+	(junction
 		(at 147.32 36.83)
 		(diameter 0)
@@
 	(wire
 		(pts
+			(xy 33.02 25.4) (xy 33.02 22.86)
+		)
+		(stroke
+			(width 0)
+			(type default)
+		)
+	)
+	(wire
+		(pts
 			(xy 134.62 76.2) (xy 134.62 67.31)
 		)
@@
 	(wire
 		(pts
-			(xy 30.48 22.86) (xy 30.48 24.13)
+			(xy 26.67 22.86) (xy 26.67 24.13)
 		)
 		(stroke
@@
 	(wire
 		(pts
+			(xy 33.02 22.86) (xy 38.1 22.86)
+		)
+		(stroke
+			(width 0)
+			(type default)
+		)
+	)
+	(wire
+		(pts
 			(xy 59.69 184.15) (xy 76.2 184.15)
 		)
@@
 	(wire
 		(pts
+			(xy 26.67 33.02) (xy 26.67 31.75)
+		)
+		(stroke
+			(width 0)
+			(type default)
+		)
+	)
+	(wire
+		(pts
 			(xy 107.95 100.33) (xy 119.38 100.33)
 		)
@@
 	(wire
 		(pts
-			(xy 22.86 22.86) (xy 30.48 22.86)
+			(xy 22.86 22.86) (xy 26.67 22.86)
 		)
 		(stroke
@@
 	(wire
 		(pts
-			(xy 30.48 22.86) (xy 38.1 22.86)
-		)
-		(stroke
-			(width 0)
-			(type default)
-		)
-	)
-	(wire
-		(pts
 			(xy 83.82 90.17) (xy 83.82 97.79)
 		)
@@
 	(wire
 		(pts
+			(xy 26.67 34.29) (xy 26.67 33.02)
+		)
+		(stroke
+			(width 0)
+			(type default)
+		)
+	)
+	(wire
+		(pts
 			(xy 227.33 100.33) (xy 233.68 100.33)
 		)
@@
 	(wire
 		(pts
+			(xy 26.67 33.02) (xy 33.02 33.02)
+		)
+		(stroke
+			(width 0)
+			(type default)
+		)
+	)
+	(wire
+		(pts
 			(xy 144.78 87.63) (xy 147.32 87.63)
 		)
@@
 	(wire
 		(pts
+			(xy 26.67 22.86) (xy 33.02 22.86)
+		)
+		(stroke
+			(width 0)
+			(type default)
+		)
+	)
+	(wire
+		(pts
 			(xy 105.41 64.77) (xy 105.41 81.28)
 		)
@@
 	(symbol
 		(lib_id "Device:C")
-		(at 30.48 27.94 0)
+		(at 26.67 27.94 0)
 		(unit 1)
 		(body_style 1)
@@
 		(in_pos_files yes)
 		(dnp no)
-		(fields_autoplaced yes)
 		(property "Reference" "C2"
-			(at 34.29 26.6699 0)
+			(at 20.574 26.162 0)
 			(show_name no)
 			(do_not_autoplace no)
@@
 		)
 		(property "Value" "2.2u"
-			(at 34.29 29.2099 0)
+			(at 19.812 28.702 0)
 			(show_name no)
 			(do_not_autoplace no)
@@
 		)
 		(property "Footprint" "Mouser:CAP_6050_TDK"
-			(at 31.4452 31.75 0)
+			(at 27.6352 31.75 0)
 			(hide yes)
 			(show_name no)
@@
 		)
 		(property "Datasheet" ""
-			(at 30.48 27.94 0)
+			(at 26.67 27.94 0)
 			(hide yes)
 			(show_name no)
@@
 		)
 		(property "Description" "Unpolarized capacitor"
-			(at 30.48 27.94 0)
+			(at 26.67 27.94 0)
+			(hide yes)
+			(show_name no)
+			(do_not_autoplace no)
+			(effects
+				(font
+					(size 1.27 1.27)
+				)
+			)
+		)
+		(property "Mouser#" "810-CAA572X6T2W225M6"
+			(at 26.67 27.94 0)
 			(hide yes)
 			(show_name no)
@@
 	(symbol
 		(lib_id "power:GNDPWR")
-		(at 30.48 31.75 0)
+		(at 26.67 34.29 0)
 		(unit 1)
 		(body_style 1)
@@
 		(fields_autoplaced yes)
 		(property "Reference" "#PWR02"
-			(at 30.48 36.83 0)
+			(at 26.67 39.37 0)
 			(hide yes)
 			(show_name no)
@@
 		)
 		(property "Value" "GNDPWR"
-			(at 30.353 35.56 0)
+			(at 26.543 38.1 0)
 			(show_name no)
 			(do_not_autoplace no)
@@
 		)
 		(property "Footprint" ""
-			(at 30.48 33.02 0)
+			(at 26.67 35.56 0)
 			(hide yes)
 			(show_name no)
@@
 		)
 		(property "Datasheet" ""
-			(at 30.48 33.02 0)
+			(at 26.67 35.56 0)
 			(hide yes)
 			(show_name no)
@@
 		)
 		(property "Description" "Power symbol creates a global label with name \"GNDPWR\" , global ground"
-			(at 30.48 31.75 0)
+			(at 26.67 34.29 0)
 			(hide yes)
 			(show_name no)
@@
 					(unit 1)
 				)
+			)
+		)
+	)
+	(symbol
+		(lib_id "Device:R_US")
+		(at 33.02 29.21 180)
+		(unit 1)
+		(body_style 1)
+		(exclude_from_sim no)
+		(in_bom yes)
+		(on_board yes)
+		(in_pos_files yes)
+		(dnp no)
+		(fields_autoplaced yes)
+		(property "Reference" "R17"
+			(at 35.56 27.9399 0)
+			(show_name no)
+			(do_not_autoplace no)
+			(effects
+				(font
+					(size 1.27 1.27)
+				)
+				(justify right)
+			)
+		)
+		(property "Value" "1.5M"
+			(at 35.56 30.4799 0)
+			(show_name no)
+			(do_not_autoplace no)
+			(effects
+				(font
+					(size 1.27 1.27)
+				)
+				(justify right)
+			)
+		)
+		(property "Footprint" "Resistor_SMD:R_2010_5025Metric_Pad1.40x2.65mm_HandSolder"
+			(at 32.004 28.956 90)
+			(hide yes)
+			(show_name no)
+			(do_not_autoplace no)
+			(effects
+				(font
+					(size 1.27 1.27)
+				)
+			)
+		)
+		(property "Datasheet" ""
+			(at 33.02 29.21 0)
+			(hide yes)
+			(show_name no)
+			(do_not_autoplace no)
+			(effects
+				(font
+					(size 1.27 1.27)
+				)
+			)
+		)
+		(property "Description" "Resistor, US symbol"
+			(at 33.02 29.21 0)
+			(hide yes)
+			(show_name no)
+			(do_not_autoplace no)
+			(effects
+				(font
+					(size 1.27 1.27)
+				)
+			)
+		)
+		(property "Mouser#" "603-RC2010JK-071M5L"
+			(at 33.02 29.21 0)
+			(hide yes)
+			(show_name no)
+			(do_not_autoplace no)
+			(effects
+				(font
+					(size 1.27 1.27)
+				)
+			)
+		)
+		(pin "1"
+		)
+		(pin "2"
+		)
+		(instances
+			(project "RML_EMO"
+				(path "/dde5c833-5196-4ddc-842a-885b47d44bef"
+					(reference "R17")
+					(unit 1)
+				)

Commit message: fixed decoupling cap issues
Parts:
- Q4: Digikey# (none) -> 5318-AM2398N-ND
- R3: Mouser# 71-CRCW0805400KJNTA -> 71-CRCW0805374KFKEA
- U7: footprint Package_TO_SOT_SMD:SOT-23-5 -> Package_TO_SOT_SMD:SOT-353_SC-70-5
Changed lines of the file:
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@@
 			)
 		)
-		(property "Datasheet" "https://www.digikey.com/en/products/detail/infineon-technologies/IPP60R180P7XKSA1/6823342?s=N4IgTCBcDaIJIAUEDYAMAlAjADlQg7ABoDSAygIKYC0AcgCKBwBAAQOIoY55FmXMCyAeVIAxAKIAVJjSoBhABJNkAVlQA1JjnJNxAsGFRUAzExABdAL5A"
+		(property "Datasheet" "https://www.digikey.com/en/products/detail/analog-power-inc/AM2398N/24883018"
 			(at 124.46 100.33 0)
 			(hide yes)
@@
 			)
 		)
-		(property "Digikey#" ""
+		(property "Digikey#" "5318-AM2398N-ND"
 			(at 124.46 100.33 0)
 			(hide yes)
@@
 			)
 		)
-		(property "Mouser#" "71-CRCW0805400KJNTA"
+		(property "Mouser#" "71-CRCW0805374KFKEA"
 			(at 68.58 104.14 0)
 			(hide yes)
@@
 			)
 		)
-		(property "Footprint" "Package_TO_SOT_SMD:SOT-23-5"
+		(property "Footprint" "Package_TO_SOT_SMD:SOT-353_SC-70-5"
 			(at 207.01 100.33 0)
 			(hide yes)

Commit message: fixed footprints and mouser# for rml
Parts:
- C1, C11: JLC# C1592 -> (none); Mouser# (none) -> 603-AC0805KKX7R9B105
- C3: JLC# C1590 -> (none); Mouser# (none) -> 603-AC0603KR9BB104
- C4, C7, C9: JLC# C91186 -> (none); Mouser# (none) -> 603-AC0805KKX7R9B105
- C6: JLC# C1591 -> (none); Mouser# (none) -> 603-AC0603KR9BB104
- R13, R15: Mouser# (none) -> 603-RC0805FR-0710KL
- R14: Mouser# (none) -> 603-RC0805FR-07680RL
- R16: Mouser# (none) -> 603-RC0805FR-10100KL
- U7: footprint Package_TO_SOT_SMD:SOT-353_SC-70-5 -> Package_TO_SOT_SMD:SOT-23-5_HandSoldering; Mouser# (none) -> 595-SN74AHC1G02DBE4
- U8: Mouser# (none) -> OPA1662DGK
Changed lines of the file:
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@@
 		(dnp no)
 		(property "Reference" "R15"
-			(at 94.996 96.012 0)
+			(at 97.917 94.869 90)
 			(show_name no)
 			(do_not_autoplace no)
@@
 		)
 		(property "Value" "10k"
-			(at 97.282 95.504 0)
+			(at 97.409 92.583 90)
 			(show_name no)
 			(do_not_autoplace no)
@@
 			)
 		)
+		(property "Mouser#" " 603-RC0805FR-0710KL "
+			(at 96.52 90.17 90)
+			(hide yes)
+			(show_name no)
+			(do_not_autoplace no)
+			(effects
+				(font
+					(size 1.27 1.27)
+				)
+			)
+		)
 		(pin "1"
 		)
@@
 			)
 		)
-		(property "JLC#" "C91186"
+		(property "JLC#" ""
+			(at 66.04 27.94 0)
+			(hide yes)
+			(show_name no)
+			(do_not_autoplace no)
+			(effects
+				(font
+					(size 1.27 1.27)
+				)
+			)
+		)
+		(property "Mouser#" " 603-AC0805KKX7R9B105 "
 			(at 66.04 27.94 0)
 			(hide yes)
@@
 			)
 		)
-		(property "JLC#" "C1592"
+		(property "JLC#" ""
+			(at 22.86 151.13 0)
+			(hide yes)
+			(show_name no)
+			(do_not_autoplace no)
+			(effects
+				(font
+					(size 1.27 1.27)
+				)
+			)
+		)
+		(property "Mouser#" " 603-AC0805KKX7R9B105 "
 			(at 22.86 151.13 0)
 			(hide yes)
@@
 			)
 		)
-		(property "JLC#" "C91186"
+		(property "JLC#" ""
 			(at 157.48 30.48 0)
 			(hide yes)
@@
 			)
 		)
+		(property "Mouser#" " 603-AC0805KKX7R9B105 "
+			(at 157.48 30.48 90)
+			(hide yes)
+			(show_name no)
+			(do_not_autoplace no)
+			(effects
+				(font
+					(size 1.27 1.27)
+				)
+			)
+		)
 		(pin "1"
 		)
@@
 			)
 		)
+		(property "Mouser#" " 603-RC0805FR-07680RL "
+			(at 223.52 100.33 90)
+			(hide yes)
+			(show_name no)
+			(do_not_autoplace no)
+			(effects
+				(font
+					(size 1.27 1.27)
+				)
+			)
+		)
 		(pin "1"
 		)
@@
 			)
 		)
-		(property "JLC#" "C1590"
+		(property "JLC#" ""
+			(at 34.29 151.13 90)
+			(hide yes)
+			(show_name no)
+			(do_not_autoplace no)
+			(effects
+				(font
+					(size 1.27 1.27)
+				)
+			)
+		)
+		(property "Mouser#" " 603-AC0603KR9BB104 "
 			(at 34.29 151.13 90)
 			(hide yes)
@@
 			)
 		)
+		(property "Mouser#" " 603-RC0805FR-0710KL "
+			(at 184.15 93.98 0)
+			(hide yes)
+			(show_name no)
+			(do_not_autoplace no)
+			(effects
+				(font
+					(size 1.27 1.27)
+				)
+			)
+		)
 		(pin "1"
 		)
@@
 			)
 		)
-		(property "JLC#" "C1592"
+		(property "JLC#" ""
+			(at 200.66 87.63 90)
+			(hide yes)
+			(show_name no)
+			(do_not_autoplace no)
+			(effects
+				(font
+					(size 1.27 1.27)
+				)
+			)
+		)
+		(property "Mouser#" " 603-AC0805KKX7R9B105 "
 			(at 200.66 87.63 90)
 			(hide yes)
@@
 			)
 		)
-		(property "JLC#" "C91186"
+		(property "JLC#" ""
+			(at 157.48 62.23 90)
+			(hide yes)
+			(show_name no)
+			(do_not_autoplace no)
+			(effects
+				(font
+					(size 1.27 1.27)
+				)
+			)
+		)
+		(property "Mouser#" " 603-AC0805KKX7R9B105 "
 			(at 157.48 62.23 90)
 			(hide yes)
@@
 			)
 		)
+		(property "Mouser#" "OPA1662DGK"
+			(at 167.64 64.77 0)
+			(hide yes)
+			(show_name no)
+			(do_not_autoplace no)
+			(effects
+				(font
+					(size 1.27 1.27)
+				)
+			)
+		)
 		(pin "5"
 		)
@@
 			)
 		)
+		(property "Mouser#" "OPA1662DGK"
+			(at 118.11 78.74 0)
+			(hide yes)
+			(show_name no)
+			(do_not_autoplace no)
+			(effects
+				(font
+					(size 1.27 1.27)
+				)
+			)
+		)
 		(pin "5"
 		)
@@
 			)
 		)
+		(property "Mouser#" "603-RC0805FR-10100KL"
+			(at 127 114.3 0)
+			(hide yes)
+			(show_name no)
+			(do_not_autoplace no)
+			(effects
+				(font
+					(size 1.27 1.27)
+				)
+			)
+		)
 		(pin "1"
 		)
@@
 			)
 		)
-		(property "Footprint" "Package_TO_SOT_SMD:SOT-353_SC-70-5"
+		(property "Footprint" "Package_TO_SOT_SMD:SOT-23-5_HandSoldering"
 			(at 207.01 100.33 0)
 			(hide yes)
@@
 			)
 		)
+		(property "Mouser#" " 595-SN74AHC1G02DBE4 "
+			(at 207.01 100.33 0)
+			(hide yes)
+			(show_name no)
+			(do_not_autoplace no)
+			(effects
+				(font
+					(size 1.27 1.27)
+				)
+			)
+		)
 		(pin "1"
 		)
@@
 			)
 		)
+		(property "Mouser#" "OPA1662DGK"
+			(at 95.25 100.33 0)
+			(hide yes)
+			(show_name no)
+			(do_not_autoplace no)
+			(effects
+				(font
+					(size 1.27 1.27)
+				)
+			)
+		)
 		(pin "5"
 		)
@@
 			)
 		)
-		(property "JLC#" "C1591"
+		(property "JLC#" ""
 			(at 114.3 31.75 0)
 			(hide yes)
@@
 			(show_name no)
 			(do_not_autoplace no)
+			(effects
+				(font
+					(size 1.27 1.27)
+				)
+			)
+		)
+		(property "Mouser#" " 603-AC0603KR9BB104 "
+			(at 114.3 31.75 90)
+			(hide yes)
+			(show_name no)
+			(do_not_autoplace no)

Commit message: added module lids and fixed RML part #s
Parts:
- C1: Manufacturer# (none) -> CC0603KRX7R9BB105
- C11, C4, C7, C9: Manufacturer# (none) -> 13-AC0805KKX7R9BB105CT-ND
- C2: Digikey# (none) -> 445-CAA572X6T2W225M640LJCT-ND; Manufacturer# (none) -> CAA572X6T2W225M640LJ; Mouser# 810-CAA572X6T2W225M6 -> (none)
- C3: Manufacturer# (none) -> 311-3034-2-ND
- C5: Mouser# 963-MLASG168BB5475KT -> 963-MLASG168BB5475KT
- C8: Manufacturer# (none) -> CC0603KRX7R6BB334; Mouser# (none) -> 603-CC603KRX7R6BB334
- D1: Manufacturer# (none) -> RFU01SM4ST2R; Mouser# 755-RFU01SM4ST2R -> 755-RFU01SM4ST2R
- D2: Mouser# 78-MMSZ5240CHE3_A-08 -> 78-MMSZ5240CHE3_A-08
- R1, R16: Digikey# (none) -> 13-RC0805FR-10100KLCT-ND; Manufacturer# (none) -> RC0805FR-10100KL; Mouser# 603-RC0805FR-10100KL -> (none)
- R10, R7: Manufacturer# (none) -> ERJ-P06F8662V
- R11: Manufacturer# (none) -> ERJ-P06J105V
- R12: Manufacturer# (none) -> ERJ-P06F6041V
- R13, R15: Digikey# (none) -> 603-RC0805FR-0710KL; Manufacturer# (none) -> 311-10.0KCRCT-ND; Mouser# 603-RC0805FR-0710KL -> (none)
- R14: Manufacturer# (none) -> RC0805FR-0710KL
- R17: Manufacturer# (none) -> CRCW20101M50FKEF
- R2: Manufacturer# (none) -> CR0805-FX-3571ELF
- R3: Manufacturer# (none) -> CRCW0805374KFKEA
- R4: Manufacturer# (none) -> ERJ-P06F3602V
- R5: Manufacturer# (none) -> RC1206FR-0747KL
- R6: Manufacturer# (none) -> RC1206FR-07100KL
- R8: Manufacturer# (none) -> ERJ-P06F1432V
- R9: Manufacturer# (none) -> CRCW08052K00JNEA
- U1: Digikey# (none) -> LR8K4-GCT-ND; Manufacturer# (none) -> LR8K4-G; Mouser# 689-LR8K4-G -> (none)
- U2: Manufacturer# (none) -> LMC555CMX/NOPBCT-ND; Mouser# (none) -> LMC555CMX/NOPB
- U5: Manufacturer# (none) -> LM1117DT-5.0/NOPB; Mouser# (none) -> 926-LM1117DT50NOPB
- U6: Manufacturer# (none) -> VOLA617A-3X001T
- U7: footprint Package_TO_SOT_SMD:SOT-23-5_HandSoldering -> Package_TO_SOT_SMD:SOT-353_SC-70-5; Manufacturer# (none) -> SN74AHC1G02DBVRE4
- U8: Manufacturer# (none) -> OPA2172QDGKRQ1

Commit message: fixed NOR gate part #
Parts:
- U7: Manufacturer# SN74AHC1G02DBVRE4 -> SN74AHC1G02DCKRG4; Mouser# 595-SN74AHC1G02DBE4 -> 595-SN74AHC1G02DCG4
Changed lines of the file:
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@@
 			)
 		)
-		(property "Mouser#" " 595-SN74AHC1G02DBE4 "
+		(property "Mouser#" "595-SN74AHC1G02DCG4"
 			(at 207.01 100.33 0)
 			(hide yes)
@@
 			)
 		)
-		(property "Manufacturer#" " SN74AHC1G02DBVRE4 "
+		(property "Manufacturer#" " SN74AHC1G02DCKRG4"
 			(at 207.01 100.33 0)
 			(hide yes)
