File: PowerBoard TR27/PowerBoard TR27.kicad_sch (KiCad schematic)
At the start: 30 parts, among them J1 Conn_01x06_Socket, J2 Conn_01x06_Socket, J3 Conn_01x01_Socket, J4 Conn_01x01_Socket, J5 Conn_01x01_Socket, J6 Conn_01x04_Socket, J7 Conn_01x04_Socket, J8 Conn_01x18_Socket, J9 Conn_01x18_Socket, Q1 Q_PMOS_DGS, Q2 Q_NMOS, U1 MC7805BDTRKG

Commit message: added mouser#
Parts:
- C3, C5: MF# (none) -> CC0603KRX7R9BB105; Mouser# (none) -> 603-CC603KRX7R9BB105
- C4, C6: MF# (none) -> CC0603KRX7R6BB334; Mouser# (none) -> 603-CC603KRX7R6BB334
- C7: MF# (none) -> 311-3034-2-ND; Mouser# (none) -> AC0603KRX7R9BB104
- D1: Digikey# 641-2082-2-ND -> (none); Mouser Price/Stock (none) -> 750-CPDUR12V-HF; Mouser# 750-CPDUR12V-HF -> 750-CPDUR12V-HF
- Q2: MF# (none) -> MMFTN6001; Mouser# (none) -> 637-MMFTN6001
- R2: MF# (none) -> ERJ-P06J105V; Mouser# (none) -> 667-ERJ-P06J105V
- R3, R4: MF# (none) -> 603-RC0805FR-0710KL; Mouser# (none) -> 603-RC0805FR-0710KL
Changed lines of the file:
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@@
 			)
 		)
+		(property "MF#" " 603-RC0805FR-0710KL  "
+			(at 194.31 43.18 0)
+			(hide yes)
+			(show_name no)
+			(do_not_autoplace no)
+			(effects
+				(font
+					(size 1.27 1.27)
+				)
+			)
+		)
+		(property "Mouser#" " 603-RC0805FR-0710KL  "
+			(at 194.31 43.18 0)
+			(hide yes)
+			(show_name no)
+			(do_not_autoplace no)
+			(effects
+				(font
+					(size 1.27 1.27)
+				)
+			)
+		)
 		(pin "1"
 		)
@@
 			)
 		)
+		(property "MF#" "CC0603KRX7R9BB105 "
+			(at 143.51 36.83 0)
+			(hide yes)
+			(show_name no)
+			(do_not_autoplace no)
+			(effects
+				(font
+					(size 1.27 1.27)
+				)
+			)
+		)
+		(property "Mouser#" "603-CC603KRX7R9BB105 "
+			(at 143.51 36.83 0)
+			(hide yes)
+			(show_name no)
+			(do_not_autoplace no)
+			(effects
+				(font
+					(size 1.27 1.27)
+				)
+			)
+		)
 		(pin "2"
 		)
@@
 			)
 		)
+		(property "MF#" "CC0603KRX7R6BB334 "
+			(at 123.19 36.83 0)
+			(hide yes)
+			(show_name no)
+			(do_not_autoplace no)
+			(effects
+				(font
+					(size 1.27 1.27)
+				)
+			)
+		)
+		(property "Mouser#" " 603-CC603KRX7R6BB334  "
+			(at 123.19 36.83 0)
+			(hide yes)
+			(show_name no)
+			(do_not_autoplace no)
+			(effects
+				(font
+					(size 1.27 1.27)
+				)
+			)
+		)
 		(pin "2"
 		)
@@
 			)
 		)
-		(property "Mouser#" " 750-CPDUR12V-HF "
+		(property "Mouser#" " 750-CPDUR12V-HF  "
 			(at 44.45 41.91 90)
 			(hide yes)
@@
 			)
 		)
-		(property "Digikey#" "641-2082-2-ND"
+		(property "Digikey#" ""
 			(at 44.45 41.91 90)
 			(hide yes)
@@
 			)
 		)
+		(property "Mouser Price/Stock" " 750-CPDUR12V-HF  "
+			(at 44.45 41.91 90)
+			(hide yes)
+			(show_name no)
+			(do_not_autoplace no)
+			(effects
+				(font
+					(size 1.27 1.27)
+				)
+			)
+		)
 		(pin "1"
 		)
@@
 			)
 		)
+		(property "MF#" "CC0603KRX7R6BB334 "
+			(at 152.4 36.83 0)
+			(hide yes)
+			(show_name no)
+			(do_not_autoplace no)
+			(effects
+				(font
+					(size 1.27 1.27)
+				)
+			)
+		)
+		(property "Mouser#" " 603-CC603KRX7R6BB334  "
+			(at 152.4 36.83 0)
+			(hide yes)
+			(show_name no)
+			(do_not_autoplace no)
+			(effects
+				(font
+					(size 1.27 1.27)
+				)
+			)
+		)
 		(pin "2"
 		)
@@
 			)
 		)
+		(property "MF#" " 603-RC0805FR-0710KL  "
+			(at 201.93 25.4 0)
+			(hide yes)
+			(show_name no)
+			(do_not_autoplace no)
+			(effects
+				(font
+					(size 1.27 1.27)
+				)
+			)
+		)
+		(property "Mouser#" " 603-RC0805FR-0710KL  "
+			(at 201.93 25.4 0)
+			(hide yes)
+			(show_name no)
+			(do_not_autoplace no)
+			(effects
+				(font
+					(size 1.27 1.27)
+				)
+			)
+		)
 		(pin "1"
 		)
@@
 			)
 		)
+		(property "MF#" " ERJ-P06J105V  "
+			(at 76.2 41.91 0)
+			(hide yes)
+			(show_name no)
+			(do_not_autoplace no)
+			(effects
+				(font
+					(size 1.27 1.27)
+				)
+			)
+		)
+		(property "Mouser#" "667-ERJ-P06J105V "
+			(at 76.2 41.91 0)
+			(hide yes)
+			(show_name no)
+			(do_not_autoplace no)
+			(effects
+				(font
+					(size 1.27 1.27)
+				)
+			)
+		)
 		(pin "1"
 		)
@@
 			)
 		)
+		(property "MF#" "311-3034-2-ND "
+			(at 163.83 36.83 0)
+			(hide yes)
+			(show_name no)
+			(do_not_autoplace no)
+			(effects
+				(font
+					(size 1.27 1.27)
+				)
+			)
+		)
+		(property "Mouser#" "AC0603KRX7R9BB104  "
+			(at 163.83 36.83 0)
+			(hide yes)
+			(show_name no)
+			(do_not_autoplace no)
+			(effects
+				(font
+					(size 1.27 1.27)
+				)
+			)
+		)
 		(pin "2"
 		)
@@
 			)
 		)
+		(property "MF#" "MMFTN6001  "
+			(at 199.39 36.83 0)
+			(hide yes)
+			(show_name no)
+			(do_not_autoplace no)
+			(effects
+				(font
+					(size 1.27 1.27)
+				)
+			)
+		)
+		(property "Mouser#" " 637-MMFTN6001  "
+			(at 199.39 36.83 0)
+			(hide yes)
+			(show_name no)
+			(do_not_autoplace no)
+			(effects
+				(font
+					(size 1.27 1.27)
+				)
+			)
+		)
 		(pin "1"
 		)
@@
 			(at 114.3 36.83 0)
 			(hide yes)
+			(show_name no)
+			(do_not_autoplace no)
+			(effects
+				(font
+					(size 1.27 1.27)
+				)
+			)
+		)
+		(property "MF#" "CC0603KRX7R9BB105 "
+			(at 114.3 36.83 0)
+			(hide yes)
+			(show_name no)
+			(do_not_autoplace no)
+			(effects
+				(font
+					(size 1.27 1.27)
+				)
+			)
+		)
+		(property "Mouser#" "603-CC603KRX7R9BB105 "
+			(at 114.3 36.83 0)
+			(hide yes)
