File: RML Constant Current/RML VERY SIMPLE/RML VERY SIMPLE.kicad_pcb (KiCad board)
At the start: 2 copper layers, 58.1 x 34 mm, 25 parts, among them J1 TE 4Pin, J2 MicroFit 4Pin, Q1 Q_NMOS_GDS, Q2 Q_NMOS_GSD, Q3 Q_NMOS_GSD, U1 NE555D, U2 Optocoupler

Commit message: small simple rml fixes
Connections:
- net HV+ renamed TS+
- D4 pad 2: HV- -> TS-
- J1 pad 2: HV- -> TS-
- Q2 pad 2: HV- -> TS-
- R5 pad 2: HV- -> TS-
Routing:
- net TS-: vias 0 -> 79
- net HV-: vias 77 -> 0
- added copper zone on B.Cu, net TS-
- added copper zone on F.Cu, net TS-
- removed copper zone on B.Cu, net HV-
- removed copper zone on F.Cu, net HV-
