File: RML Constant Current/RML VERY SIMPLE/RML VERY SIMPLE.kicad_sch (KiCad schematic)
At the start: 21 parts, among them J1 TE 4Pin, J2 MicroFit 4Pin, Q1 Q_NMOS_GDS, Q2 Q_NMOS_GSD, Q3 Q_NMOS_GSD, U1 NE555D, U2 Optocoupler

Commit message: small simple rml fixes
Connections:
- net HV-: no longer D4.2 (A), J1.2 (Pin_2), Q2.2 (S), R5.2
- net HV+ renamed TS+
- new net TS-: D4.2 (A), J1.2 (Pin_2), Q2.2 (S), R5.2
Other:
- moved on the sheet: C1, C2, C3, D1, D2, D3, D4, J1, J2, Q1, Q2, Q3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
